File: expansion.sch (KiCad schematic (older format))
At the start: 4 parts, among them P1 EXPANSION BUS

Commit message: Add RTC
Parts:
- P1: footprint MODULE -> (none)
Changed lines of the file:
@@
 $Descr A4 11693 8268
 encoding utf-8
-Sheet 11 12
+Sheet 11 13
 Title "Rämixx500"
 Date "2019-04-20"
@@
 F 0 "P1" H 5715 6065 50  0000 C CNN
 F 1 "EXPANSION BUS" H 5715 5974 50  0000 C CNN
-F 2 "MODULE" H 5715 3600 50  0001 C CNN
+F 2 "" H 5715 3600 50  0001 C CNN
 F 3 "DOCUMENTATION" H 5715 3600 50  0001 C CNN
 	1    5715 3600

Commit message: Replace RAM with original design
Parts:
- P1: footprint (none) -> Raemixx500:A2000_COPRO_SLOT
Changed lines of the file:
@@
 F 0 "P1" H 5715 6065 50  0000 C CNN
 F 1 "EXPANSION BUS" H 5715 5974 50  0000 C CNN
-F 2 "" H 5715 3600 50  0001 C CNN
+F 2 "Raemixx500:A2000_COPRO_SLOT" H 5715 3600 50  0001 C CNN
 F 3 "DOCUMENTATION" H 5715 3600 50  0001 C CNN
 	1    5715 3600

Commit message: Almost all components positioned
Parts:
- E702, E703, E704: footprint (none) -> Raemixx500:EMI_Filter_Short
Changed lines of the file:
@@
 F 0 "E702" H 7765 1220 50  0000 C CNN
 F 1 "10n" H 7575 990 50  0000 C CNN
-F 2 "" V 7765 1020 50  0001 C CNN
+F 2 "Raemixx500:EMI_Filter_Short" V 7765 1020 50  0001 C CNN
 F 3 "http://www.murata.com/~/media/webrenewal/support/library/catalog/products/emc/emifil/c31e.ashx?la=en-gb" V 7765 1020 50  0001 C CNN
 	1    7765 1020
@@
 F 0 "E703" H 7765 1855 50  0000 C CNN
 F 1 "10n" H 7575 1620 50  0000 C CNN
-F 2 "" V 7765 1650 50  0001 C CNN
+F 2 "Raemixx500:EMI_Filter_Short" V 7765 1650 50  0001 C CNN
 F 3 "http://www.murata.com/~/media/webrenewal/support/library/catalog/products/emc/emifil/c31e.ashx?la=en-gb" V 7765 1650 50  0001 C CNN
 	1    7765 1650
@@
 F 0 "E704" H 7765 2200 50  0000 C CNN
 F 1 "10n" H 7575 1970 50  0000 C CNN
-F 2 "" V 7765 2000 50  0001 C CNN
+F 2 "Raemixx500:EMI_Filter_Short" V 7765 2000 50  0001 C CNN
 F 3 "http://www.murata.com/~/media/webrenewal/support/library/catalog/products/emc/emifil/c31e.ashx?la=en-gb" V 7765 2000 50  0001 C CNN
 	1    7765 2000

Commit message: Work in progress
Connections:
- net GND: now also E702.2
Changed lines of the file:
@@
 ~HLT
+Wire Wire Line
+	7765 1070 7765 1115
+Wire Wire Line
+	7765 1115 7405 1115
+Wire Wire Line
+	7405 1115 7405 1745
 Wire Wire Line
 	3800 3000 4965 3000
@@
 Wire Bus Line
 	7155 760  7155 4200
+Connection ~ 7405 1745
 $EndSCHEMATC
