File: expansion.sch (KiCad schematic (older format))
At the start: 4 parts, among them P1 EXPANSION BUS

Commit message: Minor corrections
Other:
- note removed: "~CONFIG"
Changed lines of the file:
@@
 Wire Wire Line
 	6465 2000 6710 2000
-Text Notes 6415 2000 0    50   ~ 0
-~CONFIG
 NoConn ~ 6465 2400
 Wire Wire Line
