File: expansion.sch (KiCad schematic (older format))
At the start: 4 parts, among them P1 EXPANSION BUS

Commit message: Begin adding part numbers
Parts:
- P1: MFG Name (none) -> SKIP; MFG Part Num (none) -> SKIP; Optional (none) -> CONN
Changed lines of the file:
@@
 F 2 "Raemixx500:A2000_COPRO_SLOT" H 5715 3600 50  0001 C CNN
 F 3 "DOCUMENTATION" H 5715 3600 50  0001 C CNN
+F 4 "SKIP" H 5715 3600 50  0001 C CNN "MFG Name"
+F 5 "SKIP" H 5715 3600 50  0001 C CNN "MFG Part Num"
+F 6 "CONN" H 5715 3600 50  0001 C CNN "Optional"
 	1    5715 3600
 	1    0    0    -1

Commit message: Add EMI filter types
Parts:
- E702, E703, E704: EMI_FILTER_TYPE (none) -> W/FERRITE
Changed lines of the file:
@@
 F 2 "Raemixx500:EMI_Filter_Short" V 7765 1020 50  0001 C CNN
 F 3 "http://www.murata.com/~/media/webrenewal/support/library/catalog/products/emc/emifil/c31e.ashx?la=en-gb" V 7765 1020 50  0001 C CNN
+F 4 "W/FERRITE" H 7765 1020 50  0001 C CNN "EMI_FILTER_TYPE"
 	1    7765 1020
 	-1   0    0    -1
@@
 F 2 "Raemixx500:EMI_Filter_Short" V 7765 1650 50  0001 C CNN
 F 3 "http://www.murata.com/~/media/webrenewal/support/library/catalog/products/emc/emifil/c31e.ashx?la=en-gb" V 7765 1650 50  0001 C CNN
+F 4 "W/FERRITE" H 7765 1650 50  0001 C CNN "EMI_FILTER_TYPE"
 	1    7765 1650
 	-1   0    0    -1
@@
 F 2 "Raemixx500:EMI_Filter_Short" V 7765 2000 50  0001 C CNN
 F 3 "http://www.murata.com/~/media/webrenewal/support/library/catalog/products/emc/emifil/c31e.ashx?la=en-gb" V 7765 2000 50  0001 C CNN
+F 4 "W/FERRITE" H 7765 2000 50  0001 C CNN "EMI_FILTER_TYPE"
 	1    7765 2000
 	-1   0    0    -1

Commit message: Add part numbers for EMI filters Not the original filters, but what seem to be suitable replacements available today
Parts:
- E702, E703, E704: Cost (none) -> 0.234; MFG Name (none) -> MURATA; MFG Part Num (none) -> DSS1NB32A151Q91A
Changed lines of the file:
@@
 F 3 "http://www.murata.com/~/media/webrenewal/support/library/catalog/products/emc/emifil/c31e.ashx?la=en-gb" V 7765 1020 50  0001 C CNN
 F 4 "W/FERRITE" H 7765 1020 50  0001 C CNN "EMI_FILTER_TYPE"
+F 5 "0.234" H 7765 1020 50  0001 C CNN "Cost"
+F 6 "MURATA" H 7765 1020 50  0001 C CNN "MFG Name"
+F 7 "DSS1NB32A151Q91A" H 7765 1020 50  0001 C CNN "MFG Part Num"
 	1    7765 1020
 	-1   0    0    -1
@@
 F 3 "http://www.murata.com/~/media/webrenewal/support/library/catalog/products/emc/emifil/c31e.ashx?la=en-gb" V 7765 1650 50  0001 C CNN
 F 4 "W/FERRITE" H 7765 1650 50  0001 C CNN "EMI_FILTER_TYPE"
+F 5 "0.234" H 7765 1650 50  0001 C CNN "Cost"
+F 6 "MURATA" H 7765 1650 50  0001 C CNN "MFG Name"
+F 7 "DSS1NB32A151Q91A" H 7765 1650 50  0001 C CNN "MFG Part Num"
 	1    7765 1650
 	-1   0    0    -1
@@
 F 3 "http://www.murata.com/~/media/webrenewal/support/library/catalog/products/emc/emifil/c31e.ashx?la=en-gb" V 7765 2000 50  0001 C CNN
 F 4 "W/FERRITE" H 7765 2000 50  0001 C CNN "EMI_FILTER_TYPE"
+F 5 "0.234" H 7765 2000 50  0001 C CNN "Cost"
+F 6 "MURATA" H 7765 2000 50  0001 C CNN "MFG Name"
+F 7 "DSS1NB32A151Q91A" H 7765 2000 50  0001 C CNN "MFG Part Num"
 	1    7765 2000
 	-1   0    0    -1

Commit message: Add EMI filter 3D models, add logo, re-add Rock Lobster (closes #15) Thanks to Szabó Zoltán and Workshopshed!
Parts:
- E702, E703, E704: MFG Part Num DSS1NB32A151Q91A -> DSS1NB32A103Q91A
Changed lines of the file:
@@
 F 5 "0.234" H 7765 1020 50  0001 C CNN "Cost"
 F 6 "MURATA" H 7765 1020 50  0001 C CNN "MFG Name"
-F 7 "DSS1NB32A151Q91A" H 7765 1020 50  0001 C CNN "MFG Part Num"
+F 7 "DSS1NB32A103Q91A" H 7765 1020 50  0001 C CNN "MFG Part Num"
 	1    7765 1020
 	-1   0    0    -1
@@
 F 5 "0.234" H 7765 1650 50  0001 C CNN "Cost"
 F 6 "MURATA" H 7765 1650 50  0001 C CNN "MFG Name"
-F 7 "DSS1NB32A151Q91A" H 7765 1650 50  0001 C CNN "MFG Part Num"
+F 7 "DSS1NB32A103Q91A" H 7765 1650 50  0001 C CNN "MFG Part Num"
 	1    7765 1650
 	-1   0    0    -1
@@
 F 5 "0.234" H 7765 2000 50  0001 C CNN "Cost"
 F 6 "MURATA" H 7765 2000 50  0001 C CNN "MFG Name"
-F 7 "DSS1NB32A151Q91A" H 7765 2000 50  0001 C CNN "MFG Part Num"
+F 7 "DSS1NB32A103Q91A" H 7765 2000 50  0001 C CNN "MFG Part Num"
 	1    7765 2000
 	-1   0    0    -1

Commit message: Rename "Optional" Field to "Section"
Parts:
- P1: Optional CONN -> (none); Section (none) -> CONN
Changed lines of the file:
@@
 F 4 "SKIP" H 5715 3600 50  0001 C CNN "MFG Name"
 F 5 "SKIP" H 5715 3600 50  0001 C CNN "MFG Part Num"
-F 6 "CONN" H 5715 3600 50  0001 C CNN "Optional"
+F 6 "CONN" H 5715 3600 50  0001 C CNN "Section"
 	1    5715 3600
 	1    0    0    -1
