File: floppy.sch (KiCad schematic (older format))
At the start: 25 parts, among them CN11 INTERNAL_FLOPPY, CN12 FLOPPY_POWER, CN14 IDE_POWER, CN15 IDE_I/F, CN5 EXTFLOPPY_DB23F, U36 74LS05, U5 GARY_5719

Commit message: Almost all components positioned
Parts:
- E611, E612, E613, E614, E615, E616, E617, E618, E619, E620, E621, E622, E623, E624, E625, E626: footprint (none) -> Raemixx500:EMI_Filter_Short
Changed lines of the file:
@@
 F 0 "E613" H 2795 5750 50  0000 C CNN
 F 1 "100p" H 2745 5530 50  0000 C CNN
-F 2 "" V 2935 5560 50  0001 C CNN
+F 2 "Raemixx500:EMI_Filter_Short" V 2935 5560 50  0001 C CNN
 F 3 "http://www.murata.com/~/media/webrenewal/support/library/catalog/products/emc/emifil/c31e.ashx?la=en-gb" V 2935 5560 50  0001 C CNN
 	1    2935 5560
@@
 F 0 "E614" H 3320 5955 50  0000 C CNN
 F 1 "100p" H 3485 5730 50  0000 C CNN
-F 2 "" V 3320 5760 50  0001 C CNN
+F 2 "Raemixx500:EMI_Filter_Short" V 3320 5760 50  0001 C CNN
 F 3 "http://www.murata.com/~/media/webrenewal/support/library/catalog/products/emc/emifil/c31e.ashx?la=en-gb" V 3320 5760 50  0001 C CNN
 	1    3320 5760
@@
 F 0 "E615" H 2795 6150 50  0000 C CNN
 F 1 "100p" H 2745 5935 50  0000 C CNN
-F 2 "" V 2935 5960 50  0001 C CNN
+F 2 "Raemixx500:EMI_Filter_Short" V 2935 5960 50  0001 C CNN
 F 3 "http://www.murata.com/~/media/webrenewal/support/library/catalog/products/emc/emifil/c31e.ashx?la=en-gb" V 2935 5960 50  0001 C CNN
 	1    2935 5960
@@
 F 0 "E616" H 3320 6355 50  0000 C CNN
 F 1 "100p" H 3490 6130 50  0000 C CNN
-F 2 "" V 3320 6160 50  0001 C CNN
+F 2 "Raemixx500:EMI_Filter_Short" V 3320 6160 50  0001 C CNN
 F 3 "http://www.murata.com/~/media/webrenewal/support/library/catalog/products/emc/emifil/c31e.ashx?la=en-gb" V 3320 6160 50  0001 C CNN
 	1    3320 6160
@@
 F 0 "E611" H 2795 4350 50  0000 C CNN
 F 1 "100p" H 2745 4130 50  0000 C CNN
-F 2 "" V 2935 4160 50  0001 C CNN
+F 2 "Raemixx500:EMI_Filter_Short" V 2935 4160 50  0001 C CNN
 F 3 "http://www.murata.com/~/media/webrenewal/support/library/catalog/products/emc/emifil/c31e.ashx?la=en-gb" V 2935 4160 50  0001 C CNN
 	1    2935 4160
@@
 F 0 "E612" H 3320 4555 50  0000 C CNN
 F 1 "100p" H 3485 4330 50  0000 C CNN
-F 2 "" V 3320 4360 50  0001 C CNN
+F 2 "Raemixx500:EMI_Filter_Short" V 3320 4360 50  0001 C CNN
 F 3 "http://www.murata.com/~/media/webrenewal/support/library/catalog/products/emc/emifil/c31e.ashx?la=en-gb" V 3320 4360 50  0001 C CNN
 	1    3320 4360
@@
 F 0 "E617" H 5215 4450 50  0000 C CNN
 F 1 "100p" H 5165 4230 50  0000 C CNN
-F 2 "" V 5355 4260 50  0001 C CNN
+F 2 "Raemixx500:EMI_Filter_Short" V 5355 4260 50  0001 C CNN
 F 3 "http://www.murata.com/~/media/webrenewal/support/library/catalog/products/emc/emifil/c31e.ashx?la=en-gb" V 5355 4260 50  0001 C CNN
 	1    5355 4260
@@
 F 0 "E618" H 4970 4655 50  0000 C CNN
 F 1 "100p" H 5135 4430 50  0000 C CNN
-F 2 "" V 4970 4460 50  0001 C CNN
+F 2 "Raemixx500:EMI_Filter_Short" V 4970 4460 50  0001 C CNN
 F 3 "http://www.murata.com/~/media/webrenewal/support/library/catalog/products/emc/emifil/c31e.ashx?la=en-gb" V 4970 4460 50  0001 C CNN
 	1    4970 4460
@@
 F 0 "E619" H 5215 4850 50  0000 C CNN
 F 1 "100p" H 5165 4635 50  0000 C CNN
-F 2 "" V 5355 4660 50  0001 C CNN
+F 2 "Raemixx500:EMI_Filter_Short" V 5355 4660 50  0001 C CNN
 F 3 "http://www.murata.com/~/media/webrenewal/support/library/catalog/products/emc/emifil/c31e.ashx?la=en-gb" V 5355 4660 50  0001 C CNN
 	1    5355 4660
@@
 F 0 "E620" H 4970 5055 50  0000 C CNN
 F 1 "100p" H 5140 4830 50  0000 C CNN
-F 2 "" V 4970 4860 50  0001 C CNN
+F 2 "Raemixx500:EMI_Filter_Short" V 4970 4860 50  0001 C CNN
 F 3 "http://www.murata.com/~/media/webrenewal/support/library/catalog/products/emc/emifil/c31e.ashx?la=en-gb" V 4970 4860 50  0001 C CNN
 	1    4970 4860
@@
 F 0 "E621" H 5215 5250 50  0000 C CNN
 F 1 "100p" H 5165 5030 50  0000 C CNN
-F 2 "" V 5355 5060 50  0001 C CNN
+F 2 "Raemixx500:EMI_Filter_Short" V 5355 5060 50  0001 C CNN
 F 3 "http://www.murata.com/~/media/webrenewal/support/library/catalog/products/emc/emifil/c31e.ashx?la=en-gb" V 5355 5060 50  0001 C CNN
 	1    5355 5060
@@
 F 0 "E622" H 4970 5455 50  0000 C CNN
 F 1 "100p" H 5135 5230 50  0000 C CNN
-F 2 "" V 4970 5260 50  0001 C CNN
+F 2 "Raemixx500:EMI_Filter_Short" V 4970 5260 50  0001 C CNN
 F 3 "http://www.murata.com/~/media/webrenewal/support/library/catalog/products/emc/emifil/c31e.ashx?la=en-gb" V 4970 5260 50  0001 C CNN
 	1    4970 5260
@@
 F 0 "E623" H 5215 5650 50  0000 C CNN
 F 1 "100p" H 5165 5435 50  0000 C CNN
-F 2 "" V 5355 5460 50  0001 C CNN
+F 2 "Raemixx500:EMI_Filter_Short" V 5355 5460 50  0001 C CNN
 F 3 "http://www.murata.com/~/media/webrenewal/support/library/catalog/products/emc/emifil/c31e.ashx?la=en-gb" V 5355 5460 50  0001 C CNN
 	1    5355 5460
@@
 F 0 "E624" H 4970 5855 50  0000 C CNN
 F 1 "100p" H 5140 5630 50  0000 C CNN
-F 2 "" V 4970 5660 50  0001 C CNN
+F 2 "Raemixx500:EMI_Filter_Short" V 4970 5660 50  0001 C CNN
 F 3 "http://www.murata.com/~/media/webrenewal/support/library/catalog/products/emc/emifil/c31e.ashx?la=en-gb" V 4970 5660 50  0001 C CNN
 	1    4970 5660
@@
 F 0 "E625" H 5215 6050 50  0000 C CNN
 F 1 "100p" H 5165 5830 50  0000 C CNN
-F 2 "" V 5355 5860 50  0001 C CNN
+F 2 "Raemixx500:EMI_Filter_Short" V 5355 5860 50  0001 C CNN
 F 3 "http://www.murata.com/~/media/webrenewal/support/library/catalog/products/emc/emifil/c31e.ashx?la=en-gb" V 5355 5860 50  0001 C CNN
 	1    5355 5860
@@
 F 0 "E626" H 4970 6255 50  0000 C CNN
 F 1 "100p" H 5135 6030 50  0000 C CNN
-F 2 "" V 4970 6060 50  0001 C CNN
+F 2 "Raemixx500:EMI_Filter_Short" V 4970 6060 50  0001 C CNN
 F 3 "http://www.murata.com/~/media/webrenewal/support/library/catalog/products/emc/emifil/c31e.ashx?la=en-gb" V 4970 6060 50  0001 C CNN
 	1    4970 6060

Commit message: Almost there :)
Parts:
- CN5: footprint Raemixx500:DB_23 -> Raemixx500:DB_23F
Changed lines of the file:
@@
 Sheet 7 14
 Title "Rämixx500"
-Date "2019-04-18"
+Date "2019-06-23"
 Rev "1git"
 Comp "SukkoPera"
@@
 F 0 "CN5" H 4145 3768 50  0000 C CNN
 F 1 "EXTFLOPPY_DB23F" H 4145 3859 50  0000 C CNN
-F 2 "Raemixx500:DB_23" H 4145 5260 50  0001 C CNN
+F 2 "Raemixx500:DB_23F" H 4145 5260 50  0001 C CNN
 F 3 " ~" H 4145 5260 50  0001 C CNN
 	1    4145 5260
