File: floppy.sch (KiCad schematic (older format))
At the start: 25 parts, among them CN11 INTERNAL_FLOPPY, CN12 FLOPPY_POWER, CN14 IDE_POWER, CN15 IDE_I/F, CN5 EXTFLOPPY_DB23F, U36 74LS05, U5 GARY_5719

Commit message: Begin adding part numbers
Parts:
- CN11, CN12, CN5: Optional (none) -> FLOPPY
- CN14, CN15: MFG Name (none) -> SKIP; MFG Part Num (none) -> SKIP
- U36: Optional (none) -> FLOPPY/RTC
- U5: Optional (none) -> CUSTOM
Changed lines of the file:
@@
 F 2 "Package_DIP:DIP-48_W15.24mm_Socket_LongPads" H 2685 2060 50  0001 C CNN
 F 3 "DOCUMENTATION" H 2685 1610 50  0001 C CNN
+F 4 "CUSTOM" H 2685 1860 50  0001 C CNN "Optional"
 	2    2685 1860
 	1    0    0    -1
@@
 F 2 "Package_DIP:DIP-14_W7.62mm_Socket_LongPads" H 3940 1560 50  0001 C CNN
 F 3 "http://www.ti.com/lit/gpn/sn74LS05" H 3940 1560 50  0001 C CNN
+F 4 "FLOPPY/RTC" H 3940 1560 50  0001 C CNN "Optional"
 	1    3940 1560
 	1    0    0    -1
@@
 F 2 "Package_DIP:DIP-14_W7.62mm_Socket_LongPads" H 3940 1960 50  0001 C CNN
 F 3 "http://www.ti.com/lit/gpn/sn74LS05" H 3940 1960 50  0001 C CNN
+F 4 "FLOPPY/RTC" H 3940 1960 50  0001 C CNN "Optional"
 	2    3940 1960
 	1    0    0    -1
@@
 F 2 "Package_DIP:DIP-14_W7.62mm_Socket_LongPads" H 3940 2360 50  0001 C CNN
 F 3 "http://www.ti.com/lit/gpn/sn74LS05" H 3940 2360 50  0001 C CNN
+F 4 "FLOPPY/RTC" H 3940 2360 50  0001 C CNN "Optional"
 	3    3940 2360
 	1    0    0    -1
@@
 F 2 "Package_DIP:DIP-14_W7.62mm_Socket_LongPads" H 3940 2760 50  0001 C CNN
 F 3 "http://www.ti.com/lit/gpn/sn74LS05" H 3940 2760 50  0001 C CNN
+F 4 "FLOPPY/RTC" H 3940 2760 50  0001 C CNN "Optional"
 	4    3940 2760
 	1    0    0    -1
@@
 F 2 "Connector_PinHeader_2.54mm:PinHeader_1x04_P2.54mm_Vertical" H 9500 2475 50  0001 C CNN
 F 3 "" H 9500 2475 50  0001 C CNN
+F 4 "FLOPPY" H 9500 2475 50  0001 C CNN "Optional"
 	1    9500 2475
 	1    0    0    -1
@@
 F 2 "Connector_PinHeader_2.54mm:PinHeader_2x17_P2.54mm_Vertical" H 6915 2250 50  0001 C CNN
 F 3 "~" H 6915 2250 50  0001 C CNN
+F 4 "FLOPPY" H 6915 2250 50  0001 C CNN "Optional"
 	1    6915 2250
 	-1   0    0    -1
@@
 F 2 "Raemixx500:DB_23F" H 4145 5260 50  0001 C CNN
 F 3 " ~" H 4145 5260 50  0001 C CNN
+F 4 "FLOPPY" H 4145 5260 50  0001 C CNN "Optional"
 	1    4145 5260
 	1    0    0    1
@@
 F 2 "Connector_PinHeader_2.54mm:PinHeader_1x04_P2.54mm_Vertical" H 9500 3550 50  0001 C CNN
 F 3 "" H 9500 3550 50  0001 C CNN
+F 4 "SKIP" H 9500 3550 50  0001 C CNN "MFG Name"
+F 5 "SKIP" H 9500 3550 50  0001 C CNN "MFG Part Num"
 	1    9500 3550
 	1    0    0    -1
@@
 F 2 "Connector_PinHeader_2.54mm:PinHeader_1x04_P2.54mm_Vertical" H 9500 4735 50  0001 C CNN
 F 3 "" H 9500 4735 50  0001 C CNN
+F 4 "SKIP" H 9500 4735 50  0001 C CNN "MFG Name"
+F 5 "SKIP" H 9500 4735 50  0001 C CNN "MFG Part Num"
 	1    9500 4735
 	1    0    0    -1

Commit message: More part numbers
Parts:
- U36: Cost (none) -> 0.668; MFG Name (none) -> TI; MFG Part Num (none) -> SN74LS05N
Changed lines of the file:
@@
 F 3 "http://www.ti.com/lit/gpn/sn74LS05" H 3940 1560 50  0001 C CNN
 F 4 "FLOPPY/RTC" H 3940 1560 50  0001 C CNN "Optional"
+F 5 "0.668" H 3940 1560 50  0001 C CNN "Cost"
+F 6 "TI" H 3940 1560 50  0001 C CNN "MFG Name"
+F 7 "SN74LS05N" H 3940 1560 50  0001 C CNN "MFG Part Num"
 	1    3940 1560
 	1    0    0    -1
@@
 F 3 "http://www.ti.com/lit/gpn/sn74LS05" H 3940 1960 50  0001 C CNN
 F 4 "FLOPPY/RTC" H 3940 1960 50  0001 C CNN "Optional"
+F 5 "0.668" H 3940 1960 50  0001 C CNN "Cost"
+F 6 "TI" H 3940 1960 50  0001 C CNN "MFG Name"
+F 7 "SN74LS05N" H 3940 1960 50  0001 C CNN "MFG Part Num"
 	2    3940 1960
 	1    0    0    -1
@@
 F 3 "http://www.ti.com/lit/gpn/sn74LS05" H 3940 2360 50  0001 C CNN
 F 4 "FLOPPY/RTC" H 3940 2360 50  0001 C CNN "Optional"
+F 5 "0.668" H 3940 2360 50  0001 C CNN "Cost"
+F 6 "TI" H 3940 2360 50  0001 C CNN "MFG Name"
+F 7 "SN74LS05N" H 3940 2360 50  0001 C CNN "MFG Part Num"
 	3    3940 2360
 	1    0    0    -1
@@
 F 3 "http://www.ti.com/lit/gpn/sn74LS05" H 3940 2760 50  0001 C CNN
 F 4 "FLOPPY/RTC" H 3940 2760 50  0001 C CNN "Optional"
+F 5 "0.668" H 3940 2760 50  0001 C CNN "Cost"
+F 6 "TI" H 3940 2760 50  0001 C CNN "MFG Name"
+F 7 "SN74LS05N" H 3940 2760 50  0001 C CNN "MFG Part Num"
 	4    3940 2760
 	1    0    0    -1

Commit message: Add EMI filter types
Parts:
- E601, E602: EMI_FILTER_TYPE (none) -> W/FERRITE
- E611, E612, E613, E614, E615, E616, E617, E618, E619, E620, E621, E622, E623, E624, E625, E626: EMI_FILTER_TYPE (none) -> NORMAL
Changed lines of the file:
@@
 F 2 "Raemixx500:EMI_Filter_Short" V 2935 5560 50  0001 C CNN
 F 3 "http://www.murata.com/~/media/webrenewal/support/library/catalog/products/emc/emifil/c31e.ashx?la=en-gb" V 2935 5560 50  0001 C CNN
+F 4 "NORMAL" H 2935 5560 50  0001 C CNN "EMI_FILTER_TYPE"
 	1    2935 5560
 	1    0    0    -1
@@
 F 2 "Raemixx500:EMI_Filter_Short" V 3320 5760 50  0001 C CNN
 F 3 "http://www.murata.com/~/media/webrenewal/support/library/catalog/products/emc/emifil/c31e.ashx?la=en-gb" V 3320 5760 50  0001 C CNN
+F 4 "NORMAL" H 3320 5760 50  0001 C CNN "EMI_FILTER_TYPE"
 	1    3320 5760
 	1    0    0    -1
@@
 F 2 "Raemixx500:EMI_Filter_Short" V 2935 5960 50  0001 C CNN
 F 3 "http://www.murata.com/~/media/webrenewal/support/library/catalog/products/emc/emifil/c31e.ashx?la=en-gb" V 2935 5960 50  0001 C CNN
+F 4 "NORMAL" H 2935 5960 50  0001 C CNN "EMI_FILTER_TYPE"
 	1    2935 5960
 	1    0    0    -1
@@
 F 2 "Raemixx500:EMI_Filter_Short" V 3320 6160 50  0001 C CNN
 F 3 "http://www.murata.com/~/media/webrenewal/support/library/catalog/products/emc/emifil/c31e.ashx?la=en-gb" V 3320 6160 50  0001 C CNN
+F 4 "NORMAL" H 3320 6160 50  0001 C CNN "EMI_FILTER_TYPE"
 	1    3320 6160
 	1    0    0    -1
@@
 F 2 "Raemixx500:EMI_Filter_Long" V 2935 6360 50  0001 C CNN
 F 3 "http://www.murata.com/~/media/webrenewal/support/library/catalog/products/emc/emifil/c31e.ashx?la=en-gb" V 2935 6360 50  0001 C CNN
+F 4 "W/FERRITE" H 2935 6360 50  0001 C CNN "EMI_FILTER_TYPE"
 	1    2935 6360
 	1    0    0    -1
@@
 F 2 "Raemixx500:EMI_Filter_Short" V 2935 4160 50  0001 C CNN
 F 3 "http://www.murata.com/~/media/webrenewal/support/library/catalog/products/emc/emifil/c31e.ashx?la=en-gb" V 2935 4160 50  0001 C CNN
+F 4 "NORMAL" H 2935 4160 50  0001 C CNN "EMI_FILTER_TYPE"
 	1    2935 4160
 	1    0    0    -1
@@
 F 2 "Raemixx500:EMI_Filter_Short" V 3320 4360 50  0001 C CNN
 F 3 "http://www.murata.com/~/media/webrenewal/support/library/catalog/products/emc/emifil/c31e.ashx?la=en-gb" V 3320 4360 50  0001 C CNN
+F 4 "NORMAL" H 3320 4360 50  0001 C CNN "EMI_FILTER_TYPE"
 	1    3320 4360
 	1    0    0    -1
@@
 F 2 "Raemixx500:EMI_Filter_Short" V 5355 4260 50  0001 C CNN
 F 3 "http://www.murata.com/~/media/webrenewal/support/library/catalog/products/emc/emifil/c31e.ashx?la=en-gb" V 5355 4260 50  0001 C CNN
+F 4 "NORMAL" H 5355 4260 50  0001 C CNN "EMI_FILTER_TYPE"
 	1    5355 4260
 	-1   0    0    -1
@@
 F 2 "Raemixx500:EMI_Filter_Short" V 4970 4460 50  0001 C CNN
 F 3 "http://www.murata.com/~/media/webrenewal/support/library/catalog/products/emc/emifil/c31e.ashx?la=en-gb" V 4970 4460 50  0001 C CNN
+F 4 "NORMAL" H 4970 4460 50  0001 C CNN "EMI_FILTER_TYPE"
 	1    4970 4460
 	-1   0    0    -1
@@
 F 2 "Raemixx500:EMI_Filter_Short" V 5355 4660 50  0001 C CNN
 F 3 "http://www.murata.com/~/media/webrenewal/support/library/catalog/products/emc/emifil/c31e.ashx?la=en-gb" V 5355 4660 50  0001 C CNN
+F 4 "NORMAL" H 5355 4660 50  0001 C CNN "EMI_FILTER_TYPE"
 	1    5355 4660
 	-1   0    0    -1
@@
 F 2 "Raemixx500:EMI_Filter_Short" V 4970 4860 50  0001 C CNN
 F 3 "http://www.murata.com/~/media/webrenewal/support/library/catalog/products/emc/emifil/c31e.ashx?la=en-gb" V 4970 4860 50  0001 C CNN
+F 4 "NORMAL" H 4970 4860 50  0001 C CNN "EMI_FILTER_TYPE"
 	1    4970 4860
 	-1   0    0    -1
@@
 F 2 "Raemixx500:EMI_Filter_Short" V 5355 5060 50  0001 C CNN
 F 3 "http://www.murata.com/~/media/webrenewal/support/library/catalog/products/emc/emifil/c31e.ashx?la=en-gb" V 5355 5060 50  0001 C CNN
+F 4 "NORMAL" H 5355 5060 50  0001 C CNN "EMI_FILTER_TYPE"
 	1    5355 5060
 	-1   0    0    -1
@@
 F 2 "Raemixx500:EMI_Filter_Short" V 4970 5260 50  0001 C CNN
 F 3 "http://www.murata.com/~/media/webrenewal/support/library/catalog/products/emc/emifil/c31e.ashx?la=en-gb" V 4970 5260 50  0001 C CNN
+F 4 "NORMAL" H 4970 5260 50  0001 C CNN "EMI_FILTER_TYPE"
 	1    4970 5260
 	-1   0    0    -1
@@
 F 2 "Raemixx500:EMI_Filter_Short" V 5355 5460 50  0001 C CNN
 F 3 "http://www.murata.com/~/media/webrenewal/support/library/catalog/products/emc/emifil/c31e.ashx?la=en-gb" V 5355 5460 50  0001 C CNN
+F 4 "NORMAL" H 5355 5460 50  0001 C CNN "EMI_FILTER_TYPE"
 	1    5355 5460
 	-1   0    0    -1
@@
 F 2 "Raemixx500:EMI_Filter_Short" V 4970 5660 50  0001 C CNN
 F 3 "http://www.murata.com/~/media/webrenewal/support/library/catalog/products/emc/emifil/c31e.ashx?la=en-gb" V 4970 5660 50  0001 C CNN
+F 4 "NORMAL" H 4970 5660 50  0001 C CNN "EMI_FILTER_TYPE"
 	1    4970 5660
 	-1   0    0    -1
@@
 F 2 "Raemixx500:EMI_Filter_Short" V 5355 5860 50  0001 C CNN
 F 3 "http://www.murata.com/~/media/webrenewal/support/library/catalog/products/emc/emifil/c31e.ashx?la=en-gb" V 5355 5860 50  0001 C CNN
+F 4 "NORMAL" H 5355 5860 50  0001 C CNN "EMI_FILTER_TYPE"
 	1    5355 5860
 	-1   0    0    -1
@@
 F 2 "Raemixx500:EMI_Filter_Short" V 4970 6060 50  0001 C CNN
 F 3 "http://www.murata.com/~/media/webrenewal/support/library/catalog/products/emc/emifil/c31e.ashx?la=en-gb" V 4970 6060 50  0001 C CNN
+F 4 "NORMAL" H 4970 6060 50  0001 C CNN "EMI_FILTER_TYPE"
 	1    4970 6060
 	-1   0    0    -1
@@
 F 2 "Raemixx500:EMI_Filter_Long" V 5355 6260 50  0001 C CNN
 F 3 "http://www.murata.com/~/media/webrenewal/support/library/catalog/products/emc/emifil/c31e.ashx?la=en-gb" V 5355 6260 50  0001 C CNN
+F 4 "W/FERRITE" H 5355 6260 50  0001 C CNN "EMI_FILTER_TYPE"
 	1    5355 6260
 	-1   0    0    -1

Commit message: Add part numbers for EMI filters Not the original filters, but what seem to be suitable replacements available today
Parts:
- E601, E602: Cost (none) -> 0.234; MFG Name (none) -> MURATA; MFG Part Num (none) -> DSS1NB32A151Q91A
- E611, E612, E613, E614, E615, E616, E617, E618, E619, E620, E621, E622, E623, E624, E625, E626: Cost (none) -> 0.233; MFG Part Num (none) -> DSS1NB32A101Q91A (has ferrite)
Changed lines of the file:
@@
 F 3 "http://www.murata.com/~/media/webrenewal/support/library/catalog/products/emc/emifil/c31e.ashx?la=en-gb" V 2935 5560 50  0001 C CNN
 F 4 "NORMAL" H 2935 5560 50  0001 C CNN "EMI_FILTER_TYPE"
+F 5 "0.233" H 2935 5560 50  0001 C CNN "Cost"
+F 6 "DSS1NB32A101Q91A (has ferrite)" H 2935 5560 50  0001 C CNN "MFG Part Num"
 	1    2935 5560
 	1    0    0    -1
@@
 F 3 "http://www.murata.com/~/media/webrenewal/support/library/catalog/products/emc/emifil/c31e.ashx?la=en-gb" V 3320 5760 50  0001 C CNN
 F 4 "NORMAL" H 3320 5760 50  0001 C CNN "EMI_FILTER_TYPE"
+F 5 "0.233" H 3320 5760 50  0001 C CNN "Cost"
+F 6 "DSS1NB32A101Q91A (has ferrite)" H 3320 5760 50  0001 C CNN "MFG Part Num"
 	1    3320 5760
 	1    0    0    -1
@@
 F 3 "http://www.murata.com/~/media/webrenewal/support/library/catalog/products/emc/emifil/c31e.ashx?la=en-gb" V 2935 5960 50  0001 C CNN
 F 4 "NORMAL" H 2935 5960 50  0001 C CNN "EMI_FILTER_TYPE"
+F 5 "0.233" H 2935 5960 50  0001 C CNN "Cost"
+F 6 "DSS1NB32A101Q91A (has ferrite)" H 2935 5960 50  0001 C CNN "MFG Part Num"
 	1    2935 5960
 	1    0    0    -1
@@
 F 3 "http://www.murata.com/~/media/webrenewal/support/library/catalog/products/emc/emifil/c31e.ashx?la=en-gb" V 3320 6160 50  0001 C CNN
 F 4 "NORMAL" H 3320 6160 50  0001 C CNN "EMI_FILTER_TYPE"
+F 5 "0.233" H 3320 6160 50  0001 C CNN "Cost"
+F 6 "DSS1NB32A101Q91A (has ferrite)" H 3320 6160 50  0001 C CNN "MFG Part Num"
 	1    3320 6160
 	1    0    0    -1
@@
 F 3 "http://www.murata.com/~/media/webrenewal/support/library/catalog/products/emc/emifil/c31e.ashx?la=en-gb" V 2935 6360 50  0001 C CNN
 F 4 "W/FERRITE" H 2935 6360 50  0001 C CNN "EMI_FILTER_TYPE"
+F 5 "0.234" H 2935 6360 50  0001 C CNN "Cost"
+F 6 "MURATA" H 2935 6360 50  0001 C CNN "MFG Name"
+F 7 "DSS1NB32A151Q91A" H 2935 6360 50  0001 C CNN "MFG Part Num"
 	1    2935 6360
 	1    0    0    -1
@@
 F 3 "http://www.murata.com/~/media/webrenewal/support/library/catalog/products/emc/emifil/c31e.ashx?la=en-gb" V 2935 4160 50  0001 C CNN
 F 4 "NORMAL" H 2935 4160 50  0001 C CNN "EMI_FILTER_TYPE"
+F 5 "0.233" H 2935 4160 50  0001 C CNN "Cost"
+F 6 "DSS1NB32A101Q91A (has ferrite)" H 2935 4160 50  0001 C CNN "MFG Part Num"
 	1    2935 4160
 	1    0    0    -1
@@
 F 3 "http://www.murata.com/~/media/webrenewal/support/library/catalog/products/emc/emifil/c31e.ashx?la=en-gb" V 3320 4360 50  0001 C CNN
 F 4 "NORMAL" H 3320 4360 50  0001 C CNN "EMI_FILTER_TYPE"
+F 5 "0.233" H 3320 4360 50  0001 C CNN "Cost"
+F 6 "DSS1NB32A101Q91A (has ferrite)" H 3320 4360 50  0001 C CNN "MFG Part Num"
 	1    3320 4360
 	1    0    0    -1
@@
 F 3 "http://www.murata.com/~/media/webrenewal/support/library/catalog/products/emc/emifil/c31e.ashx?la=en-gb" V 5355 4260 50  0001 C CNN
 F 4 "NORMAL" H 5355 4260 50  0001 C CNN "EMI_FILTER_TYPE"
+F 5 "0.233" H 5355 4260 50  0001 C CNN "Cost"
+F 6 "DSS1NB32A101Q91A (has ferrite)" H 5355 4260 50  0001 C CNN "MFG Part Num"
 	1    5355 4260
 	-1   0    0    -1
@@
 F 3 "http://www.murata.com/~/media/webrenewal/support/library/catalog/products/emc/emifil/c31e.ashx?la=en-gb" V 4970 4460 50  0001 C CNN
 F 4 "NORMAL" H 4970 4460 50  0001 C CNN "EMI_FILTER_TYPE"
+F 5 "0.233" H 4970 4460 50  0001 C CNN "Cost"
+F 6 "DSS1NB32A101Q91A (has ferrite)" H 4970 4460 50  0001 C CNN "MFG Part Num"
 	1    4970 4460
 	-1   0    0    -1
@@
 F 3 "http://www.murata.com/~/media/webrenewal/support/library/catalog/products/emc/emifil/c31e.ashx?la=en-gb" V 5355 4660 50  0001 C CNN
 F 4 "NORMAL" H 5355 4660 50  0001 C CNN "EMI_FILTER_TYPE"
+F 5 "0.233" H 5355 4660 50  0001 C CNN "Cost"
+F 6 "DSS1NB32A101Q91A (has ferrite)" H 5355 4660 50  0001 C CNN "MFG Part Num"
 	1    5355 4660
 	-1   0    0    -1
@@
 F 3 "http://www.murata.com/~/media/webrenewal/support/library/catalog/products/emc/emifil/c31e.ashx?la=en-gb" V 4970 4860 50  0001 C CNN
 F 4 "NORMAL" H 4970 4860 50  0001 C CNN "EMI_FILTER_TYPE"
+F 5 "0.233" H 4970 4860 50  0001 C CNN "Cost"
+F 6 "DSS1NB32A101Q91A (has ferrite)" H 4970 4860 50  0001 C CNN "MFG Part Num"
 	1    4970 4860
 	-1   0    0    -1
@@
 F 3 "http://www.murata.com/~/media/webrenewal/support/library/catalog/products/emc/emifil/c31e.ashx?la=en-gb" V 5355 5060 50  0001 C CNN
 F 4 "NORMAL" H 5355 5060 50  0001 C CNN "EMI_FILTER_TYPE"
+F 5 "0.233" H 5355 5060 50  0001 C CNN "Cost"
+F 6 "DSS1NB32A101Q91A (has ferrite)" H 5355 5060 50  0001 C CNN "MFG Part Num"
 	1    5355 5060
 	-1   0    0    -1
@@
 F 3 "http://www.murata.com/~/media/webrenewal/support/library/catalog/products/emc/emifil/c31e.ashx?la=en-gb" V 4970 5260 50  0001 C CNN
 F 4 "NORMAL" H 4970 5260 50  0001 C CNN "EMI_FILTER_TYPE"
+F 5 "0.233" H 4970 5260 50  0001 C CNN "Cost"
+F 6 "DSS1NB32A101Q91A (has ferrite)" H 4970 5260 50  0001 C CNN "MFG Part Num"
 	1    4970 5260
 	-1   0    0    -1
@@
 F 3 "http://www.murata.com/~/media/webrenewal/support/library/catalog/products/emc/emifil/c31e.ashx?la=en-gb" V 5355 5460 50  0001 C CNN
 F 4 "NORMAL" H 5355 5460 50  0001 C CNN "EMI_FILTER_TYPE"
+F 5 "0.233" H 5355 5460 50  0001 C CNN "Cost"
+F 6 "DSS1NB32A101Q91A (has ferrite)" H 5355 5460 50  0001 C CNN "MFG Part Num"
 	1    5355 5460
 	-1   0    0    -1
@@
 F 3 "http://www.murata.com/~/media/webrenewal/support/library/catalog/products/emc/emifil/c31e.ashx?la=en-gb" V 4970 5660 50  0001 C CNN
 F 4 "NORMAL" H 4970 5660 50  0001 C CNN "EMI_FILTER_TYPE"
+F 5 "0.233" H 4970 5660 50  0001 C CNN "Cost"
+F 6 "DSS1NB32A101Q91A (has ferrite)" H 4970 5660 50  0001 C CNN "MFG Part Num"
 	1    4970 5660
 	-1   0    0    -1
@@
 F 3 "http://www.murata.com/~/media/webrenewal/support/library/catalog/products/emc/emifil/c31e.ashx?la=en-gb" V 5355 5860 50  0001 C CNN
 F 4 "NORMAL" H 5355 5860 50  0001 C CNN "EMI_FILTER_TYPE"
+F 5 "0.233" H 5355 5860 50  0001 C CNN "Cost"
+F 6 "DSS1NB32A101Q91A (has ferrite)" H 5355 5860 50  0001 C CNN "MFG Part Num"
 	1    5355 5860
 	-1   0    0    -1
@@
 F 3 "http://www.murata.com/~/media/webrenewal/support/library/catalog/products/emc/emifil/c31e.ashx?la=en-gb" V 4970 6060 50  0001 C CNN
 F 4 "NORMAL" H 4970 6060 50  0001 C CNN "EMI_FILTER_TYPE"
+F 5 "0.233" H 4970 6060 50  0001 C CNN "Cost"
+F 6 "DSS1NB32A101Q91A (has ferrite)" H 4970 6060 50  0001 C CNN "MFG Part Num"
 	1    4970 6060
 	-1   0    0    -1
@@
 F 3 "http://www.murata.com/~/media/webrenewal/support/library/catalog/products/emc/emifil/c31e.ashx?la=en-gb" V 5355 6260 50  0001 C CNN
 F 4 "W/FERRITE" H 5355 6260 50  0001 C CNN "EMI_FILTER_TYPE"
+F 5 "0.234" H 5355 6260 50  0001 C CNN "Cost"
+F 6 "MURATA" H 5355 6260 50  0001 C CNN "MFG Name"
+F 7 "DSS1NB32A151Q91A" H 5355 6260 50  0001 C CNN "MFG Part Num"
 	1    5355 6260
 	-1   0    0    -1

Commit message: Add EMI filter 3D models, add logo, re-add Rock Lobster (closes #15) Thanks to Szabó Zoltán and Workshopshed!
Parts:
- E601, E602: MFG Part Num DSS1NB32A151Q91A -> DSS1NB32A103Q91A
Changed lines of the file:
@@
 F 5 "0.234" H 2935 6360 50  0001 C CNN "Cost"
 F 6 "MURATA" H 2935 6360 50  0001 C CNN "MFG Name"
-F 7 "DSS1NB32A151Q91A" H 2935 6360 50  0001 C CNN "MFG Part Num"
+F 7 "DSS1NB32A103Q91A" H 2935 6360 50  0001 C CNN "MFG Part Num"
 	1    2935 6360
 	1    0    0    -1
@@
 F 5 "0.234" H 5355 6260 50  0001 C CNN "Cost"
 F 6 "MURATA" H 5355 6260 50  0001 C CNN "MFG Name"
-F 7 "DSS1NB32A151Q91A" H 5355 6260 50  0001 C CNN "MFG Part Num"
+F 7 "DSS1NB32A103Q91A" H 5355 6260 50  0001 C CNN "MFG Part Num"
 	1    5355 6260
 	-1   0    0    -1

Commit message: Use full IDC connector for floppy and some cosmetic fixes
Parts:
- CN11: footprint Connector_PinHeader_2.54mm:PinHeader_2x17_P2.54mm_Vertical -> Connector_IDC:IDC-Header_2x17_P2.54mm_Vertical
Changed lines of the file:
@@
 F 0 "CN11" H 6965 3267 50  0000 C CNN
 F 1 "INTERNAL_FLOPPY" H 6965 3176 50  0000 C CNN
-F 2 "Connector_PinHeader_2.54mm:PinHeader_2x17_P2.54mm_Vertical" H 6915 2250 50  0001 C CNN
+F 2 "Connector_IDC:IDC-Header_2x17_P2.54mm_Vertical" H 6915 2250 50  0001 C CNN
 F 3 "~" H 6915 2250 50  0001 C CNN
 F 4 "FLOPPY" H 6915 2250 50  0001 C CNN "Optional"

Commit message: (Try to) Identify the minimum set of required components
Parts:
- U5: Required (none) -> Y
Changed lines of the file:
@@
 F 3 "DOCUMENTATION" H 2685 1610 50  0001 C CNN
 F 4 "CUSTOM" H 2685 1860 50  0001 C CNN "Optional"
+F 5 "Y" H 2685 1860 50  0001 C CNN "Required"
 	2    2685 1860
 	1    0    0    -1

Commit message: Rename "Optional" Field to "Section"
Parts:
- CN11, CN12, CN5: Optional FLOPPY -> (none); Section (none) -> FLOPPY
- U36: Optional FLOPPY/RTC -> (none); Section (none) -> FLOPPY/RTC
- U5: Optional CUSTOM -> (none); Section (none) -> CUSTOM
Changed lines of the file:
@@
 F 2 "Package_DIP:DIP-48_W15.24mm_Socket_LongPads" H 2685 2060 50  0001 C CNN
 F 3 "DOCUMENTATION" H 2685 1610 50  0001 C CNN
-F 4 "CUSTOM" H 2685 1860 50  0001 C CNN "Optional"
+F 4 "CUSTOM" H 2685 1860 50  0001 C CNN "Section"
 F 5 "Y" H 2685 1860 50  0001 C CNN "Required"
 	2    2685 1860
@@
 F 2 "Package_DIP:DIP-14_W7.62mm_Socket_LongPads" H 3940 1560 50  0001 C CNN
 F 3 "http://www.ti.com/lit/gpn/sn74LS05" H 3940 1560 50  0001 C CNN
-F 4 "FLOPPY/RTC" H 3940 1560 50  0001 C CNN "Optional"
+F 4 "FLOPPY/RTC" H 3940 1560 50  0001 C CNN "Section"
 F 5 "0.668" H 3940 1560 50  0001 C CNN "Cost"
 F 6 "TI" H 3940 1560 50  0001 C CNN "MFG Name"
@@
 F 2 "Package_DIP:DIP-14_W7.62mm_Socket_LongPads" H 3940 1960 50  0001 C CNN
 F 3 "http://www.ti.com/lit/gpn/sn74LS05" H 3940 1960 50  0001 C CNN
-F 4 "FLOPPY/RTC" H 3940 1960 50  0001 C CNN "Optional"
+F 4 "FLOPPY/RTC" H 3940 1960 50  0001 C CNN "Section"
 F 5 "0.668" H 3940 1960 50  0001 C CNN "Cost"
 F 6 "TI" H 3940 1960 50  0001 C CNN "MFG Name"
@@
 F 2 "Package_DIP:DIP-14_W7.62mm_Socket_LongPads" H 3940 2360 50  0001 C CNN
 F 3 "http://www.ti.com/lit/gpn/sn74LS05" H 3940 2360 50  0001 C CNN
-F 4 "FLOPPY/RTC" H 3940 2360 50  0001 C CNN "Optional"
+F 4 "FLOPPY/RTC" H 3940 2360 50  0001 C CNN "Section"
 F 5 "0.668" H 3940 2360 50  0001 C CNN "Cost"
 F 6 "TI" H 3940 2360 50  0001 C CNN "MFG Name"
@@
 F 2 "Package_DIP:DIP-14_W7.62mm_Socket_LongPads" H 3940 2760 50  0001 C CNN
 F 3 "http://www.ti.com/lit/gpn/sn74LS05" H 3940 2760 50  0001 C CNN
-F 4 "FLOPPY/RTC" H 3940 2760 50  0001 C CNN "Optional"
+F 4 "FLOPPY/RTC" H 3940 2760 50  0001 C CNN "Section"
 F 5 "0.668" H 3940 2760 50  0001 C CNN "Cost"
 F 6 "TI" H 3940 2760 50  0001 C CNN "MFG Name"
@@
 F 2 "Connector_PinHeader_2.54mm:PinHeader_1x04_P2.54mm_Vertical" H 9500 2475 50  0001 C CNN
 F 3 "" H 9500 2475 50  0001 C CNN
-F 4 "FLOPPY" H 9500 2475 50  0001 C CNN "Optional"
+F 4 "FLOPPY" H 9500 2475 50  0001 C CNN "Section"
 	1    9500 2475
 	1    0    0    -1
@@
 F 2 "Connector_IDC:IDC-Header_2x17_P2.54mm_Vertical" H 6915 2250 50  0001 C CNN
 F 3 "~" H 6915 2250 50  0001 C CNN
-F 4 "FLOPPY" H 6915 2250 50  0001 C CNN "Optional"
+F 4 "FLOPPY" H 6915 2250 50  0001 C CNN "Section"
 	1    6915 2250
 	-1   0    0    -1
@@
 F 2 "Raemixx500:DB_23F" H 4145 5260 50  0001 C CNN
 F 3 " ~" H 4145 5260 50  0001 C CNN
-F 4 "FLOPPY" H 4145 5260 50  0001 C CNN "Optional"
+F 4 "FLOPPY" H 4145 5260 50  0001 C CNN "Section"
 	1    4145 5260
 	1    0    0    1
