File: cpu.sch (KiCad schematic (older format))
At the start: 26 parts, among them U1 68000D, U10 74LS244, U11 74LS373, U12 74LS244, U13 74LS373, U2 FAT_AGNUS_8375, U33 74LS258, U37 74LS32, U5 GARY_5719, X1 XTAL

Commit message: Begin adding part numbers
Parts:
- C99: Cost (none) -> 0.035; MFG Name (none) -> AVX; MFG Part Num (none) -> SA115C104KAR
- E666: Cost (none) -> 0.141; MFG Name (none) -> AVX; MFG Part Num (none) -> SA102A220JARC; Optional (none) -> CLOCK
- FB101, FB102, R103, R104, R105, R106, R107, U33, X1: Optional (none) -> CLOCK
- JP2: MFG Name (none) -> SKIP; MFG Part Num (none) -> SKIP; Optional (none) -> JMP
- R101, R111, R112, R114, U10, U11, U12, U13: Optional (none) -> MEMORY
- U1: Optional (none) -> CPU
- U2, U5: Optional (none) -> CUSTOM
- U37: Optional (none) -> PARALLEL/FLOPPY/KEYBOARD
Changed lines of the file:
@@
 F 2 "Raemixx500:R_Axial_DIN0309_L9.0mm_D3.2mm_P12.70mm_Horizontal" V 13160 2800 50  0001 C CNN
 F 3 "~" H 13230 2800 50  0001 C CNN
+F 4 "MEMORY" H 13230 2800 50  0001 C CNN "Optional"
 	1    13230 2800
 	0    1    1    0
@@
 F 2 "Package_LCC:PLCC-84_THT-Socket" H 11480 7485 50  0001 C CNN
 F 3 "DOCUMENTATION" H 11480 7485 50  0001 C CNN
+F 4 "CUSTOM" H 11480 7485 50  0001 C CNN "Optional"
 	1    11480 7485
 	1    0    0    -1
@@
 F 2 "Raemixx500:R_Axial_DIN0309_L9.0mm_D3.2mm_P12.70mm_Horizontal" V 11610 4745 50  0001 C CNN
 F 3 "~" H 11680 4745 50  0001 C CNN
+F 4 "CLOCK" H 11680 4745 50  0001 C CNN "Optional"
 	1    11680 4745
 	1    0    0    -1
@@
 F 2 "Raemixx500:R_Axial_DIN0309_L9.0mm_D3.2mm_P12.70mm_Horizontal" V 11810 4745 50  0001 C CNN
 F 3 "~" H 11880 4745 50  0001 C CNN
+F 4 "CLOCK" H 11880 4745 50  0001 C CNN "Optional"
 	1    11880 4745
 	1    0    0    -1
@@
 F 2 "Raemixx500:R_Axial_DIN0309_L9.0mm_D3.2mm_P12.70mm_Horizontal" V 12010 4745 50  0001 C CNN
 F 3 "~" H 12080 4745 50  0001 C CNN
+F 4 "CLOCK" H 12080 4745 50  0001 C CNN "Optional"
 	1    12080 4745
 	1    0    0    -1
@@
 F 2 "Package_DIP:DIP-14_W7.62mm_Socket_LongPads" H 13200 4120 50  0001 C CNN
 F 3 "http://www.ti.com/lit/gpn/sn74LS32" H 13200 4120 50  0001 C CNN
+F 4 "PARALLEL/FLOPPY/KEYBOARD" H 13200 4120 50  0001 C CNN "Optional"
 	1    13200 4120
 	1    0    0    -1
@@
 F 2 "Package_DIP:DIP-14_W7.62mm_Socket_LongPads" H 13200 4455 50  0001 C CNN
 F 3 "http://www.ti.com/lit/gpn/sn74LS32" H 13200 4455 50  0001 C CNN
+F 4 "PARALLEL/FLOPPY/KEYBOARD" H 13200 4455 50  0001 C CNN "Optional"
 	2    13200 4455
 	1    0    0    -1
@@
 F 2 "Raemixx500:Jumper3-Bridged23" H 9900 4885 50  0001 C CNN
 F 3 "~" H 9900 4885 50  0001 C CNN
+F 4 "SKIP" H 9900 4885 50  0001 C CNN "MFG Name"
+F 5 "SKIP" H 9900 4885 50  0001 C CNN "MFG Part Num"
+F 6 "JMP" H 9900 4885 50  0001 C CNN "Optional"
 	1    9900 4885
 	0    -1   1    0
@@
 F 2 "Raemixx500:R_Axial_DIN0309_L9.0mm_D3.2mm_P12.70mm_Horizontal" V 13325 8635 50  0001 C CNN
 F 3 "~" H 13395 8635 50  0001 C CNN
+F 4 "CLOCK" H 13395 8635 50  0001 C CNN "Optional"
 	1    13395 8635
 	0    1    1    0
@@
 F 2 "Raemixx500:R_Axial_DIN0309_L9.0mm_D3.2mm_P12.70mm_Horizontal" V 13325 8495 50  0001 C CNN
 F 3 "~" H 13395 8495 50  0001 C CNN
+F 4 "CLOCK" H 13395 8495 50  0001 C CNN "Optional"
 	1    13395 8495
 	0    1    1    0
@@
 F 2 "Raemixx500:C_Axial_L6.3mm_D2.5mm_P10.16mm" H 14513 8465 50  0001 C CNN
 F 3 "~" H 14475 8615 50  0001 C CNN
+F 4 "0.035" H 14475 8615 50  0001 C CNN "Cost"
+F 5 "AVX" H 14475 8615 50  0001 C CNN "MFG Name"
+F 6 "SA115C104KAR" H 14475 8615 50  0001 C CNN "MFG Part Num"
 	1    14475 8615
 	1    0    0    -1
@@
 F 2 "Raemixx500:R_Axial_DIN0309_L9.0mm_D3.2mm_P12.70mm_Horizontal" V 9780 3200 50  0001 C CNN
 F 3 "~" H 9850 3200 50  0001 C CNN
+F 4 "MEMORY" H 9850 3200 50  0001 C CNN "Optional"
 	1    9850 3200
 	0    1    1    0
@@
 F 2 "Package_DIP:DIP-64_W22.86mm_Socket_LongPads" H 3635 4635 50  0001 C CNN
 F 3 "https://www.nxp.com/docs/en/reference-manual/MC68000UM.pdf" H 3635 4635 50  0001 C CNN
+F 4 "CPU" H 3635 4635 50  0001 C CNN "Optional"
 	1    3635 4635
 	1    0    0    -1
@@
 F 2 "Package_DIP:DIP-20_W7.62mm_Socket_LongPads" H 6775 3835 50  0001 C CNN
 F 3 "http://www.ti.com/lit/gpn/sn74LS373" H 6775 3835 50  0001 C CNN
+F 4 "MEMORY" H 6775 3835 50  0001 C CNN "Optional"
 	1    6775 3835
 	-1   0    0    1
@@
 F 2 "Package_DIP:DIP-20_W7.62mm_Socket_LongPads" H 6775 6635 50  0001 C CNN
 F 3 "http://www.ti.com/lit/gpn/sn74LS373" H 6775 6635 50  0001 C CNN
+F 4 "MEMORY" H 6775 6635 50  0001 C CNN "Optional"
 	1    6775 6635
 	-1   0    0    1
@@
 F 2 "Raemixx500:R_Axial_DIN0309_L9.0mm_D3.2mm_P12.70mm_Horizontal" V 9200 1150 50  0001 C CNN
 F 3 "~" H 9270 1150 50  0001 C CNN
+F 4 "MEMORY" H 9270 1150 50  0001 C CNN "Optional"
 	1    9270 1150
 	0    1    1    0
@@
 F 2 "Raemixx500:R_Axial_DIN0309_L9.0mm_D3.2mm_P12.70mm_Horizontal" V 9200 1250 50  0001 C CNN
 F 3 "~" H 9270 1250 50  0001 C CNN
+F 4 "MEMORY" H 9270 1250 50  0001 C CNN "Optional"
 	1    9270 1250
 	0    1    1    0
@@
 F 2 "Package_DIP:DIP-20_W7.62mm_Socket_LongPads" H 6775 5230 50  0001 C CNN
 F 3 "http://www.ti.com/lit/gpn/sn74LS244" H 6775 5230 50  0001 C CNN
+F 4 "MEMORY" H 6775 5230 50  0001 C CNN "Optional"
 	1    6775 5230
 	1    0    0    1
@@
 F 2 "Package_DIP:DIP-20_W7.62mm_Socket_LongPads" H 6775 2425 50  0001 C CNN
 F 3 "http://www.ti.com/lit/gpn/sn74LS244" H 6775 2425 50  0001 C CNN
+F 4 "MEMORY" H 6775 2425 50  0001 C CNN "Optional"
 	1    6775 2425
 	1    0    0    1
@@
 F 2 "Package_DIP:DIP-48_W15.24mm_Socket_LongPads" H 11480 2650 50  0001 C CNN
 F 3 "DOCUMENTATION" H 11480 2200 50  0001 C CNN
+F 4 "CUSTOM" H 11480 2450 50  0001 C CNN "Optional"
 	1    11480 2450
 	1    0    0    -1
@@
 F 2 "Package_DIP:DIP-16_W7.62mm_Socket_LongPads" H 11710 7960 50  0001 C CNN
 F 3 "http://www.ti.com/lit/gpn/sn74LS258" H 11710 7960 50  0001 C CNN
+F 4 "CLOCK" H 8610 10260 50  0001 C CNN "Optional"
 	4    8610 10260
 	1    0    0    -1
@@
 F 2 "Raemixx500:C_Axial_L6.3mm_D2.5mm_P10.16mm" H 9970 10470 50  0001 C CNN
 F 3 "~" H 9970 10470 50  0001 C CNN
+F 4 "0.141" H 9970 10470 50  0001 C CNN "Cost"
+F 5 "AVX" H 9970 10470 50  0001 C CNN "MFG Name"
+F 6 "SA102A220JARC" H 9970 10470 50  0001 C CNN "MFG Part Num"
+F 7 "CLOCK" H 9970 10470 50  0001 C CNN "Optional"
 	1    9970 10470
 	1    0    0    -1
@@
 F 2 "Oscillator:Oscillator_DIP-14" H 7150 9610 50  0001 C CNN
 F 3 "http://www.txccorp.com/download/products/osc/7C_o.pdf" H 6950 10260 50  0001 C CNN
+F 4 "CLOCK" H 7050 10260 50  0001 C CNN "Optional"
 	1    7050 10260
 	1    0    0    -1
@@
 F 2 "Raemixx500:EMI_Filter_Long" V 7740 10260 50  0001 C CNN
 F 3 "http://www.murata.com/~/media/webrenewal/support/library/catalog/products/emc/emifil/c31e.ashx?la=en-gb" V 7740 10260 50  0001 C CNN
+F 4 "CLOCK" H 7740 10260 50  0001 C CNN "Optional"
 	1    7740 10260
 	1    0    0    -1
@@
 F 2 "Raemixx500:EMI_Filter_Long" V 9395 10360 50  0001 C CNN
 F 3 "http://www.murata.com/~/media/webrenewal/support/library/catalog/products/emc/emifil/c31e.ashx?la=en-gb" V 9395 10360 50  0001 C CNN
+F 4 "CLOCK" H 9395 10360 50  0001 C CNN "Optional"
 	1    9395 10360
 	1    0    0    -1

Commit message: More part numbers
Parts:
- U10, U12: Cost (none) -> 0.62; MFG Name (none) -> TI; MFG Part Num (none) -> SN74LS244N
- U11, U13: Cost (none) -> 0.68; MFG Name (none) -> TI; MFG Part Num (none) -> SN74LS373N
- U33: MFG Name (none) -> N/A
- U37: Cost (none) -> 0.442; MFG Name (none) -> TI; MFG Part Num (none) -> SN74LS32N
Changed lines of the file:
@@
 F 3 "http://www.ti.com/lit/gpn/sn74LS32" H 13200 4120 50  0001 C CNN
 F 4 "PARALLEL/FLOPPY/KEYBOARD" H 13200 4120 50  0001 C CNN "Optional"
+F 5 "0.442" H 13200 4120 50  0001 C CNN "Cost"
+F 6 "TI" H 13200 4120 50  0001 C CNN "MFG Name"
+F 7 "SN74LS32N" H 13200 4120 50  0001 C CNN "MFG Part Num"
 	1    13200 4120
 	1    0    0    -1
@@
 F 3 "http://www.ti.com/lit/gpn/sn74LS32" H 13200 4455 50  0001 C CNN
 F 4 "PARALLEL/FLOPPY/KEYBOARD" H 13200 4455 50  0001 C CNN "Optional"
+F 5 "0.442" H 13200 4455 50  0001 C CNN "Cost"
+F 6 "TI" H 13200 4455 50  0001 C CNN "MFG Name"
+F 7 "SN74LS32N" H 13200 4455 50  0001 C CNN "MFG Part Num"
 	2    13200 4455
 	1    0    0    -1
@@
 F 3 "http://www.ti.com/lit/gpn/sn74LS373" H 6775 3835 50  0001 C CNN
 F 4 "MEMORY" H 6775 3835 50  0001 C CNN "Optional"
+F 5 "0.68" H 6775 3835 50  0001 C CNN "Cost"
+F 6 "TI" H 6775 3835 50  0001 C CNN "MFG Name"
+F 7 "SN74LS373N" H 6775 3835 50  0001 C CNN "MFG Part Num"
 	1    6775 3835
 	-1   0    0    1
@@
 F 3 "http://www.ti.com/lit/gpn/sn74LS373" H 6775 6635 50  0001 C CNN
 F 4 "MEMORY" H 6775 6635 50  0001 C CNN "Optional"
+F 5 "0.68" H 6775 6635 50  0001 C CNN "Cost"
+F 6 "TI" H 6775 6635 50  0001 C CNN "MFG Name"
+F 7 "SN74LS373N" H 6775 6635 50  0001 C CNN "MFG Part Num"
 	1    6775 6635
 	-1   0    0    1
@@
 F 3 "http://www.ti.com/lit/gpn/sn74LS244" H 6775 5230 50  0001 C CNN
 F 4 "MEMORY" H 6775 5230 50  0001 C CNN "Optional"
+F 5 "0.62" H 6775 5230 50  0001 C CNN "Cost"
+F 6 "TI" H 6775 5230 50  0001 C CNN "MFG Name"
+F 7 "SN74LS244N" H 6775 5230 50  0001 C CNN "MFG Part Num"
 	1    6775 5230
 	1    0    0    1
@@
 F 3 "http://www.ti.com/lit/gpn/sn74LS244" H 6775 2425 50  0001 C CNN
 F 4 "MEMORY" H 6775 2425 50  0001 C CNN "Optional"
+F 5 "0.62" H 6775 2425 50  0001 C CNN "Cost"
+F 6 "TI" H 6775 2425 50  0001 C CNN "MFG Name"
+F 7 "SN74LS244N" H 6775 2425 50  0001 C CNN "MFG Part Num"
 	1    6775 2425
 	1    0    0    1
@@
 F 3 "http://www.ti.com/lit/gpn/sn74LS258" H 11710 7960 50  0001 C CNN
 F 4 "CLOCK" H 8610 10260 50  0001 C CNN "Optional"
+F 5 "N/A" H 8610 10260 50  0001 C CNN "MFG Name"
 	4    8610 10260
 	1    0    0    -1

Commit message: Add EMI filter types
Parts:
- E666: EMI_FILTER_TYPE (none) -> C
- FB101, FB102: EMI_FILTER_TYPE (none) -> R
Changed lines of the file:
@@
 F 6 "SA102A220JARC" H 9970 10470 50  0001 C CNN "MFG Part Num"
 F 7 "CLOCK" H 9970 10470 50  0001 C CNN "Optional"
+F 8 "C" H 9970 10470 50  0001 C CNN "EMI_FILTER_TYPE"
 	1    9970 10470
 	1    0    0    -1
@@
 F 3 "http://www.murata.com/~/media/webrenewal/support/library/catalog/products/emc/emifil/c31e.ashx?la=en-gb" V 7740 10260 50  0001 C CNN
 F 4 "CLOCK" H 7740 10260 50  0001 C CNN "Optional"
+F 5 "R" H 7740 10260 50  0001 C CNN "EMI_FILTER_TYPE"
 	1    7740 10260
 	1    0    0    -1
@@
 F 3 "http://www.murata.com/~/media/webrenewal/support/library/catalog/products/emc/emifil/c31e.ashx?la=en-gb" V 9395 10360 50  0001 C CNN
 F 4 "CLOCK" H 9395 10360 50  0001 C CNN "Optional"
+F 5 "R" H 9395 10360 50  0001 C CNN "EMI_FILTER_TYPE"
 	1    9395 10360
 	1    0    0    -1

Commit message: (Try to) Identify the minimum set of required components
Parts:
- E666: Required (none) -> R
- FB101, FB102, R101, R102, R103, R104, R105, R106, R107, R111, R112, R113, R114, U1, U10, U11, U12, U13, U2, U33, U37, U5, X1: Required (none) -> Y
Changed lines of the file:
@@
 F 3 "~" H 13230 2800 50  0001 C CNN
 F 4 "MEMORY" H 13230 2800 50  0001 C CNN "Optional"
+F 5 "Y" H 13230 2800 50  0001 C CNN "Required"
 	1    13230 2800
 	0    1    1    0
@@
 F 3 "DOCUMENTATION" H 11480 7485 50  0001 C CNN
 F 4 "CUSTOM" H 11480 7485 50  0001 C CNN "Optional"
+F 5 "Y" H 11480 7485 50  0001 C CNN "Required"
 	1    11480 7485
 	1    0    0    -1
@@
 F 3 "~" H 11680 4745 50  0001 C CNN
 F 4 "CLOCK" H 11680 4745 50  0001 C CNN "Optional"
+F 5 "Y" H 11680 4745 50  0001 C CNN "Required"
 	1    11680 4745
 	1    0    0    -1
@@
 F 3 "~" H 11880 4745 50  0001 C CNN
 F 4 "CLOCK" H 11880 4745 50  0001 C CNN "Optional"
+F 5 "Y" H 11880 4745 50  0001 C CNN "Required"
 	1    11880 4745
 	1    0    0    -1
@@
 F 3 "~" H 12080 4745 50  0001 C CNN
 F 4 "CLOCK" H 12080 4745 50  0001 C CNN "Optional"
+F 5 "Y" H 12080 4745 50  0001 C CNN "Required"
 	1    12080 4745
 	1    0    0    -1
@@
 F 6 "TI" H 13200 4120 50  0001 C CNN "MFG Name"
 F 7 "SN74LS32N" H 13200 4120 50  0001 C CNN "MFG Part Num"
+F 8 "Y" H 13200 4120 50  0001 C CNN "Required"
 	1    13200 4120
 	1    0    0    -1
@@
 F 6 "TI" H 13200 4455 50  0001 C CNN "MFG Name"
 F 7 "SN74LS32N" H 13200 4455 50  0001 C CNN "MFG Part Num"
+F 8 "Y" H 13200 4455 50  0001 C CNN "Required"
 	2    13200 4455
 	1    0    0    -1
@@
 F 3 "~" H 13395 8635 50  0001 C CNN
 F 4 "CLOCK" H 13395 8635 50  0001 C CNN "Optional"
+F 5 "Y" H 13395 8635 50  0001 C CNN "Required"
 	1    13395 8635
 	0    1    1    0
@@
 F 3 "~" H 13395 8495 50  0001 C CNN
 F 4 "CLOCK" H 13395 8495 50  0001 C CNN "Optional"
+F 5 "Y" H 13395 8495 50  0001 C CNN "Required"
 	1    13395 8495
 	0    1    1    0
@@
 F 3 "~" H 9850 3200 50  0001 C CNN
 F 4 "MEMORY" H 9850 3200 50  0001 C CNN "Optional"
+F 5 "Y" H 9850 3200 50  0001 C CNN "Required"
 	1    9850 3200
 	0    1    1    0
@@
 F 2 "Raemixx500:R_Axial_DIN0309_L9.0mm_D3.2mm_P12.70mm_Horizontal" V 9205 2350 50  0001 C CNN
 F 3 "~" H 9275 2350 50  0001 C CNN
+F 4 "Y" H 9275 2350 50  0001 C CNN "Required"
 	1    9275 2350
 	0    1    1    0
@@
 F 3 "https://www.nxp.com/docs/en/reference-manual/MC68000UM.pdf" H 3635 4635 50  0001 C CNN
 F 4 "CPU" H 3635 4635 50  0001 C CNN "Optional"
+F 5 "Y" H 3635 4635 50  0001 C CNN "Required"
 	1    3635 4635
 	1    0    0    -1
@@
 F 6 "TI" H 6775 3835 50  0001 C CNN "MFG Name"
 F 7 "SN74LS373N" H 6775 3835 50  0001 C CNN "MFG Part Num"
+F 8 "Y" H 6775 3835 50  0001 C CNN "Required"
 	1    6775 3835
 	-1   0    0    1
@@
 F 6 "TI" H 6775 6635 50  0001 C CNN "MFG Name"
 F 7 "SN74LS373N" H 6775 6635 50  0001 C CNN "MFG Part Num"
+F 8 "Y" H 6775 6635 50  0001 C CNN "Required"
 	1    6775 6635
 	-1   0    0    1
@@
 F 2 "Raemixx500:R_Axial_DIN0309_L9.0mm_D3.2mm_P12.70mm_Horizontal" V 9200 1050 50  0001 C CNN
 F 3 "~" H 9270 1050 50  0001 C CNN
+F 4 "Y" H 9270 1050 50  0001 C CNN "Required"
 	1    9270 1050
 	0    1    1    0
@@
 F 3 "~" H 9270 1150 50  0001 C CNN
 F 4 "MEMORY" H 9270 1150 50  0001 C CNN "Optional"
+F 5 "Y" H 9270 1150 50  0001 C CNN "Required"
 	1    9270 1150
 	0    1    1    0
@@
 F 3 "~" H 9270 1250 50  0001 C CNN
 F 4 "MEMORY" H 9270 1250 50  0001 C CNN "Optional"
+F 5 "Y" H 9270 1250 50  0001 C CNN "Required"
 	1    9270 1250
 	0    1    1    0
@@
 F 6 "TI" H 6775 5230 50  0001 C CNN "MFG Name"
 F 7 "SN74LS244N" H 6775 5230 50  0001 C CNN "MFG Part Num"
+F 8 "Y" H 6775 5230 50  0001 C CNN "Required"
 	1    6775 5230
 	1    0    0    1
@@
 F 6 "TI" H 6775 2425 50  0001 C CNN "MFG Name"
 F 7 "SN74LS244N" H 6775 2425 50  0001 C CNN "MFG Part Num"
+F 8 "Y" H 6775 2425 50  0001 C CNN "Required"
 	1    6775 2425
 	1    0    0    1
@@
 F 3 "DOCUMENTATION" H 11480 2200 50  0001 C CNN
 F 4 "CUSTOM" H 11480 2450 50  0001 C CNN "Optional"
+F 5 "Y" H 11480 2450 50  0001 C CNN "Required"
 	1    11480 2450
 	1    0    0    -1
@@
 F 4 "CLOCK" H 8610 10260 50  0001 C CNN "Optional"
 F 5 "N/A" H 8610 10260 50  0001 C CNN "MFG Name"
+F 6 "Y" H 8610 10260 50  0001 C CNN "Required"
 	4    8610 10260
 	1    0    0    -1
@@
 F 7 "CLOCK" H 9970 10470 50  0001 C CNN "Optional"
 F 8 "C" H 9970 10470 50  0001 C CNN "EMI_FILTER_TYPE"
+F 9 "R" H 9970 10470 50  0001 C CNN "Required"
 	1    9970 10470
 	1    0    0    -1
@@
 F 3 "http://www.txccorp.com/download/products/osc/7C_o.pdf" H 6950 10260 50  0001 C CNN
 F 4 "CLOCK" H 7050 10260 50  0001 C CNN "Optional"
+F 5 "Y" H 7050 10260 50  0001 C CNN "Required"
 	1    7050 10260
 	1    0    0    -1
@@
 F 4 "CLOCK" H 7740 10260 50  0001 C CNN "Optional"
 F 5 "R" H 7740 10260 50  0001 C CNN "EMI_FILTER_TYPE"
+F 6 "Y" H 7740 10260 50  0001 C CNN "Required"
 	1    7740 10260
 	1    0    0    -1
@@
 F 4 "CLOCK" H 9395 10360 50  0001 C CNN "Optional"
 F 5 "R" H 9395 10360 50  0001 C CNN "EMI_FILTER_TYPE"
+F 6 "Y" H 9395 10360 50  0001 C CNN "Required"
 	1    9395 10360
 	1    0    0    -1
