File: audio.sch (KiCad schematic (older format))
At the start: 94 parts, among them CN1 LEFT_JOY, CN2 RIGHT_JOY, CN3 RIGHT, CN4 LEFT, Q301 2N3906, Q321 MPF102, Q331 MPF102, U14 LF347, U15 74LS157, U3 PAULA, U38 MC1488

Commit message: Begin adding part numbers
Parts:
- C15, C308: Cost (none) -> 0.071; MFG Name (none) -> KEMET; MFG Part Num (none) -> C410C103K1H5TAAUTO
- C3, C301, C302, C305, C325, C335: Cost (none) -> 0.078; MFG Name (none) -> KEMET; MFG Part Num (none) -> C412C334M5U5TA
- C311, C312, C313, C314: Cost (none) -> 0.284; MFG Name (none) -> KEMET; MFG Part Num (none) -> C410C473M5U5TA
- C321, C331: Cost (none) -> 0.035; MFG Name (none) -> AVX; MFG Part Num (none) -> SA115C104KAR
- C322, C332: MFG Name (none) -> KEMET; MFG Part Num (none) -> C430C682J5G5TA
- C323, C333: MFG Name (none) -> N/A
- C411, C412, C413, C421, C422, C423: Cost (none) -> 0.083; MFG Name (none) -> AVX; MFG Part Num (none) -> SA101C102KAR
- CN1, CN2, U15: Optional (none) -> JOYSTICK
- CN3, CN4, U14: Optional (none) -> AUDIO
- JP10A1, JP10B1, JP8: MFG Name (none) -> SKIP; MFG Part Num (none) -> SKIP; Optional (none) -> JMP
- U3: Optional (none) -> CUSTOM
- U38: Optional (none) -> SERIAL

Commit message: Use D12.5mm for C307 as well
Parts:
- C307: footprint Capacitor_THT:CP_Radial_D8.0mm_P5.00mm -> Capacitor_THT:CP_Radial_D12.5mm_P5.00mm
Changed lines of the file:
@@
 F 0 "C307" H 2360 2161 50  0000 L CNN
 F 1 "1000u" H 2360 2070 50  0000 L CNN
-F 2 "Capacitor_THT:CP_Radial_D8.0mm_P5.00mm" H 2245 2115 50  0001 C CNN
+F 2 "Capacitor_THT:CP_Radial_D12.5mm_P5.00mm" H 2245 2115 50  0001 C CNN
 F 3 "~" H 2245 2115 50  0001 C CNN
 	1    2245 2115

Commit message: More part numbers
Parts:
- C303, C304, C324, C334: Cost (none) -> 0.118; MFG Name (none) -> PANASONIC; MFG Part Num (none) -> EEUFR1H220
- C306: Cost (none) -> 0.196; MFG Name (none) -> PANASONIC; MFG Part Num (none) -> EEUFR1H100
- C307: Cost (none) -> 0.343; MFG Name (none) -> PANASONIC; MFG Part Num (none) -> EEUFR1C102
- U14: Cost (none) -> 0.58; MFG Name (none) -> TI; MFG Part Num (none) -> LF347N ???
- U15: Cost (none) -> 0.236; MFG Name (none) -> TI; MFG Part Num (none) -> SN74HCT157NE4
- U38: Cost (none) -> 0.615; MFG Name (none) -> TI; MFG Part Num (none) -> MC1488N
Changed lines of the file:
@@
 F 3 "http://www.ti.com/lit/gpn/sn74LS157" H 12455 3375 50  0001 C CNN
 F 4 "JOYSTICK" H 12455 3375 50  0001 C CNN "Optional"
+F 5 "0.236" H 12455 3375 50  0001 C CNN "Cost"
+F 6 "TI" H 12455 3375 50  0001 C CNN "MFG Name"
+F 7 "SN74HCT157NE4" H 12455 3375 50  0001 C CNN "MFG Part Num"
 	1    12455 3375
 	1    0    0    -1
@@
 F 3 "http://www.ti.com/lit/ds/symlink/tl081.pdf" H 9615 9115 50  0001 C CNN
 F 4 "AUDIO" H 9565 8915 50  0001 C CNN "Optional"
+F 5 "0.58" H 9565 8915 50  0001 C CNN "Cost"
+F 6 "TI" H 9565 8915 50  0001 C CNN "MFG Name"
+F 7 "LF347N ???" H 9565 8915 50  0001 C CNN "MFG Part Num"
 	1    9565 8915
 	1    0    0    -1
@@
 F 3 "http://www.ti.com/lit/ds/symlink/tl081.pdf" H 9615 7320 50  0001 C CNN
 F 4 "AUDIO" H 9565 7120 50  0001 C CNN "Optional"
+F 5 "0.58" H 9565 7120 50  0001 C CNN "Cost"
+F 6 "TI" H 9565 7120 50  0001 C CNN "MFG Name"
+F 7 "LF347N ???" H 9565 7120 50  0001 C CNN "MFG Part Num"
 	2    9565 7120
 	1    0    0    -1
@@
 F 3 "http://www.ti.com/lit/ds/symlink/tl081.pdf" H 7665 7220 50  0001 C CNN
 F 4 "AUDIO" H 7615 7020 50  0001 C CNN "Optional"
+F 5 "0.58" H 7615 7020 50  0001 C CNN "Cost"
+F 6 "TI" H 7615 7020 50  0001 C CNN "MFG Name"
+F 7 "LF347N ???" H 7615 7020 50  0001 C CNN "MFG Part Num"
 	3    7615 7020
 	1    0    0    1
@@
 F 3 "http://www.ti.com/lit/ds/symlink/tl081.pdf" H 7665 9015 50  0001 C CNN
 F 4 "AUDIO" H 7615 8815 50  0001 C CNN "Optional"
+F 5 "0.58" H 7615 8815 50  0001 C CNN "Cost"
+F 6 "TI" H 7615 8815 50  0001 C CNN "MFG Name"
+F 7 "LF347N ???" H 7615 8815 50  0001 C CNN "MFG Part Num"
 	4    7615 8815
 	1    0    0    1
@@
 F 2 "Capacitor_THT:CP_Radial_D8.0mm_P5.00mm" H 10475 9035 50  0001 C CNN
 F 3 "~" H 10475 9035 50  0001 C CNN
+F 4 "0.118" H 10475 9035 50  0001 C CNN "Cost"
+F 5 "PANASONIC" H 10475 9035 50  0001 C CNN "MFG Name"
+F 6 "EEUFR1H220" H 10475 9035 50  0001 C CNN "MFG Part Num"
 	1    10475 9035
 	0    -1   -1   0
@@
 F 2 "Capacitor_THT:CP_Radial_D8.0mm_P5.00mm" H 10475 7240 50  0001 C CNN
 F 3 "~" H 10475 7240 50  0001 C CNN
+F 4 "0.118" H 10475 7240 50  0001 C CNN "Cost"
+F 5 "PANASONIC" H 10475 7240 50  0001 C CNN "MFG Name"
+F 6 "EEUFR1H220" H 10475 7240 50  0001 C CNN "MFG Part Num"
 	1    10475 7240
 	0    -1   -1   0
@@
 F 3 "DOCUMENTATION" H 3835 9285 50  0001 C CNN
 F 4 "SERIAL" H 3835 9285 50  0001 C CNN "Optional"
+F 5 "0.615" H 3835 9285 50  0001 C CNN "Cost"
+F 6 "TI" H 3835 9285 50  0001 C CNN "MFG Name"
+F 7 "MC1488N" H 3835 9285 50  0001 C CNN "MFG Part Num"
 	1    3835 9285
 	1    0    0    -1
@@
 F 3 "http://www.ti.com/lit/ds/symlink/tl081.pdf" H 1340 9905 50  0001 C CNN
 F 4 "AUDIO" H 1290 9705 50  0001 C CNN "Optional"
+F 5 "0.58" H 1290 9705 50  0001 C CNN "Cost"
+F 6 "TI" H 1290 9705 50  0001 C CNN "MFG Name"
+F 7 "LF347N ???" H 1290 9705 50  0001 C CNN "MFG Part Num"
 	5    1290 9705
 	1    0    0    -1
@@
 F 2 "Capacitor_THT:CP_Radial_D12.5mm_P5.00mm" H 2245 2115 50  0001 C CNN
 F 3 "~" H 2245 2115 50  0001 C CNN
+F 4 "0.343" H 2245 2115 50  0001 C CNN "Cost"
+F 5 "PANASONIC" H 2245 2115 50  0001 C CNN "MFG Name"
+F 6 "EEUFR1C102" H 2245 2115 50  0001 C CNN "MFG Part Num"
 	1    2245 2115
 	1    0    0    -1
@@
 F 2 "Capacitor_THT:CP_Radial_D5.0mm_P2.50mm" H 4265 2115 50  0001 C CNN
 F 3 "~" H 4265 2115 50  0001 C CNN
+F 4 "0.196" H 4265 2115 50  0001 C CNN "Cost"
+F 5 "PANASONIC" H 4265 2115 50  0001 C CNN "MFG Name"
+F 6 "EEUFR1H100" H 4265 2115 50  0001 C CNN "MFG Part Num"
 	1    4265 2115
 	1    0    0    -1
@@
 F 2 "Capacitor_THT:CP_Radial_D5.0mm_P2.50mm" H 2060 9515 50  0001 C CNN
 F 3 "~" H 2060 9515 50  0001 C CNN
+F 4 "0.118" H 2060 9515 50  0001 C CNN "Cost"
+F 5 "PANASONIC" H 2060 9515 50  0001 C CNN "MFG Name"
+F 6 "EEUFR1H220" H 2060 9515 50  0001 C CNN "MFG Part Num"
 	1    2060 9515
 	1    0    0    -1
@@
 F 2 "Capacitor_THT:CP_Radial_D5.0mm_P2.50mm" H 2060 9900 50  0001 C CNN
 F 3 "~" H 2060 9900 50  0001 C CNN
+F 4 "0.118" H 2060 9900 50  0001 C CNN "Cost"
+F 5 "PANASONIC" H 2060 9900 50  0001 C CNN "MFG Name"
+F 6 "EEUFR1H220" H 2060 9900 50  0001 C CNN "MFG Part Num"
 	1    2060 9900
 	1    0    0    -1
@@
 F 3 "http://www.ti.com/lit/gpn/sn74LS157" H 14900 3345 50  0001 C CNN
 F 4 "JOYSTICK" H 14900 3345 50  0001 C CNN "Optional"
+F 5 "0.236" H 14900 3345 50  0001 C CNN "Cost"
+F 6 "TI" H 14900 3345 50  0001 C CNN "MFG Name"
+F 7 "SN74HCT157NE4" H 14900 3345 50  0001 C CNN "MFG Part Num"
 	2    14900 3345
 	1    0    0    -1

Commit message: Add EMI filter types
Parts:
- E302, E303, E305, E306, E415, E416, E417, E425, E426, E427, E441, E442, E443, E444: EMI_FILTER_TYPE (none) -> W/FERRITE
- E401, E408, E411, E412, E413, E414, E421, E422, E423, E424: EMI_FILTER_TYPE (none) -> W/FERRITE; Optional (none) -> JOYSTICK
- FB802: EMI_FILTER_TYPE (none) -> FERRITE
Changed lines of the file:
@@
 F 2 "Raemixx500:Ferrite_Axial_L9.0mm_D3.2mm_P12.70mm" V 4260 8070 50  0001 C CNN
 F 3 "~" H 4330 8070 50  0001 C CNN
+F 4 "FERRITE" H 4330 8070 50  0001 C CNN "EMI_FILTER_TYPE"
 	1    4330 8070
 	1    0    0    -1
@@
 F 2 "Raemixx500:EMI_Filter_Long" V 7090 2700 50  0001 C CNN
 F 3 "http://www.murata.com/~/media/webrenewal/support/library/catalog/products/emc/emifil/c31e.ashx?la=en-gb" V 7090 2700 50  0001 C CNN
+F 4 "W/FERRITE" H 7090 2700 50  0001 C CNN "EMI_FILTER_TYPE"
 	1    7090 2700
 	1    0    0    -1
@@
 F 2 "Raemixx500:EMI_Filter_Long" V 7580 2900 50  0001 C CNN
 F 3 "http://www.murata.com/~/media/webrenewal/support/library/catalog/products/emc/emifil/c31e.ashx?la=en-gb" V 7580 2900 50  0001 C CNN
+F 4 "W/FERRITE" H 7580 2900 50  0001 C CNN "EMI_FILTER_TYPE"
 	1    7580 2900
 	1    0    0    -1
@@
 F 2 "Raemixx500:EMI_Filter_Long" V 7090 4330 50  0001 C CNN
 F 3 "http://www.murata.com/~/media/webrenewal/support/library/catalog/products/emc/emifil/c31e.ashx?la=en-gb" V 7090 4330 50  0001 C CNN
+F 4 "W/FERRITE" H 7090 4330 50  0001 C CNN "EMI_FILTER_TYPE"
 	1    7090 4330
 	1    0    0    -1
@@
 F 2 "Raemixx500:EMI_Filter_Long" V 7580 5130 50  0001 C CNN
 F 3 "http://www.murata.com/~/media/webrenewal/support/library/catalog/products/emc/emifil/c31e.ashx?la=en-gb" V 7580 5130 50  0001 C CNN
+F 4 "W/FERRITE" H 7580 5130 50  0001 C CNN "EMI_FILTER_TYPE"
 	1    7580 5130
 	1    0    0    -1
@@
 F 2 "Raemixx500:EMI_Filter_Long" V 9645 1685 50  0001 C CNN
 F 3 "http://www.murata.com/~/media/webrenewal/support/library/catalog/products/emc/emifil/c31e.ashx?la=en-gb" V 9645 1685 50  0001 C CNN
+F 4 "W/FERRITE" H 9645 1685 50  0001 C CNN "EMI_FILTER_TYPE"
+F 5 "JOYSTICK" H 9645 1685 50  0001 C CNN "Optional"
 	1    9645 1685
 	-1   0    0    -1
@@
 F 2 "Raemixx500:EMI_Filter_Long" V 9645 2115 50  0001 C CNN
 F 3 "http://www.murata.com/~/media/webrenewal/support/library/catalog/products/emc/emifil/c31e.ashx?la=en-gb" V 9645 2115 50  0001 C CNN
+F 4 "W/FERRITE" H 9645 2115 50  0001 C CNN "EMI_FILTER_TYPE"
+F 5 "JOYSTICK" H 9645 2115 50  0001 C CNN "Optional"
 	1    9645 2115
 	-1   0    0    -1
@@
 F 2 "Raemixx500:EMI_Filter_Long" V 9645 2515 50  0001 C CNN
 F 3 "http://www.murata.com/~/media/webrenewal/support/library/catalog/products/emc/emifil/c31e.ashx?la=en-gb" V 9645 2515 50  0001 C CNN
+F 4 "W/FERRITE" H 9645 2515 50  0001 C CNN "EMI_FILTER_TYPE"
+F 5 "JOYSTICK" H 9645 2515 50  0001 C CNN "Optional"
 	1    9645 2515
 	-1   0    0    -1
@@
 F 2 "Raemixx500:EMI_Filter_Long" V 9645 3915 50  0001 C CNN
 F 3 "http://www.murata.com/~/media/webrenewal/support/library/catalog/products/emc/emifil/c31e.ashx?la=en-gb" V 9645 3915 50  0001 C CNN
+F 4 "W/FERRITE" H 9645 3915 50  0001 C CNN "EMI_FILTER_TYPE"
+F 5 "JOYSTICK" H 9645 3915 50  0001 C CNN "Optional"
 	1    9645 3915
 	-1   0    0    -1
@@
 F 2 "Raemixx500:EMI_Filter_Long" V 9645 4345 50  0001 C CNN
 F 3 "http://www.murata.com/~/media/webrenewal/support/library/catalog/products/emc/emifil/c31e.ashx?la=en-gb" V 9645 4345 50  0001 C CNN
+F 4 "W/FERRITE" H 9645 4345 50  0001 C CNN "EMI_FILTER_TYPE"
+F 5 "JOYSTICK" H 9645 4345 50  0001 C CNN "Optional"
 	1    9645 4345
 	-1   0    0    -1
@@
 F 2 "Raemixx500:EMI_Filter_Long" V 9645 5165 50  0001 C CNN
 F 3 "http://www.murata.com/~/media/webrenewal/support/library/catalog/products/emc/emifil/c31e.ashx?la=en-gb" V 9645 5165 50  0001 C CNN
+F 4 "W/FERRITE" H 9645 5165 50  0001 C CNN "EMI_FILTER_TYPE"
+F 5 "JOYSTICK" H 9645 5165 50  0001 C CNN "Optional"
 	1    9645 5165
 	-1   0    0    -1
@@
 F 2 "Raemixx500:EMI_Filter_Long" V 13420 2680 50  0001 C CNN
 F 3 "http://www.murata.com/~/media/webrenewal/support/library/catalog/products/emc/emifil/c31e.ashx?la=en-gb" V 13420 2680 50  0001 C CNN
+F 4 "W/FERRITE" H 13420 2680 50  0001 C CNN "EMI_FILTER_TYPE"
 	1    13420 2680
 	1    0    0    -1
@@
 F 2 "Raemixx500:EMI_Filter_Long" V 13420 3110 50  0001 C CNN
 F 3 "http://www.murata.com/~/media/webrenewal/support/library/catalog/products/emc/emifil/c31e.ashx?la=en-gb" V 13420 3110 50  0001 C CNN
+F 4 "W/FERRITE" H 13420 3110 50  0001 C CNN "EMI_FILTER_TYPE"
 	1    13420 3110
 	1    0    0    -1
@@
 F 2 "Raemixx500:EMI_Filter_Long" V 13420 3510 50  0001 C CNN
 F 3 "http://www.murata.com/~/media/webrenewal/support/library/catalog/products/emc/emifil/c31e.ashx?la=en-gb" V 13420 3510 50  0001 C CNN
+F 4 "W/FERRITE" H 13420 3510 50  0001 C CNN "EMI_FILTER_TYPE"
 	1    13420 3510
 	1    0    0    -1
@@
 F 2 "Raemixx500:EMI_Filter_Long" V 13420 3930 50  0001 C CNN
 F 3 "http://www.murata.com/~/media/webrenewal/support/library/catalog/products/emc/emifil/c31e.ashx?la=en-gb" V 13420 3930 50  0001 C CNN
+F 4 "W/FERRITE" H 13420 3930 50  0001 C CNN "EMI_FILTER_TYPE"
 	1    13420 3930
 	1    0    0    -1
@@
 F 2 "Raemixx500:EMI_Filter_Long" V 6310 7020 50  0001 C CNN
 F 3 "http://www.murata.com/~/media/webrenewal/support/library/catalog/products/emc/emifil/c31e.ashx?la=en-gb" V 6310 7020 50  0001 C CNN
+F 4 "W/FERRITE" H 6310 7020 50  0001 C CNN "EMI_FILTER_TYPE"
 	1    6310 7020
 	1    0    0    -1
@@
 F 2 "Raemixx500:EMI_Filter_Long" V 6310 8815 50  0001 C CNN
 F 3 "http://www.murata.com/~/media/webrenewal/support/library/catalog/products/emc/emifil/c31e.ashx?la=en-gb" V 6310 8815 50  0001 C CNN
+F 4 "W/FERRITE" H 6310 8815 50  0001 C CNN "EMI_FILTER_TYPE"
 	1    6310 8815
 	1    0    0    -1
@@
 F 2 "Raemixx500:EMI_Filter_Short" V 12020 9015 50  0001 C CNN
 F 3 "http://www.murata.com/~/media/webrenewal/support/library/catalog/products/emc/emifil/c31e.ashx?la=en-gb" V 12020 9015 50  0001 C CNN
+F 4 "W/FERRITE" H 12020 9015 50  0001 C CNN "EMI_FILTER_TYPE"
 	1    12020 9015
 	1    0    0    -1
@@
 F 2 "Raemixx500:EMI_Filter_Short" V 12020 7220 50  0001 C CNN
 F 3 "http://www.murata.com/~/media/webrenewal/support/library/catalog/products/emc/emifil/c31e.ashx?la=en-gb" V 12020 7220 50  0001 C CNN
+F 4 "W/FERRITE" H 12020 7220 50  0001 C CNN "EMI_FILTER_TYPE"
 	1    12020 7220
 	1    0    0    -1
@@
 F 2 "Raemixx500:EMI_Filter_Long" V 9645 2935 50  0001 C CNN
 F 3 "http://www.murata.com/~/media/webrenewal/support/library/catalog/products/emc/emifil/c31e.ashx?la=en-gb" V 9645 2935 50  0001 C CNN
+F 4 "W/FERRITE" H 9645 2935 50  0001 C CNN "EMI_FILTER_TYPE"
+F 5 "JOYSTICK" H 9645 2935 50  0001 C CNN "Optional"
 	1    9645 2935
 	-1   0    0    -1
@@
 F 2 "Raemixx500:EMI_Filter_Long" V 9645 4745 50  0001 C CNN
 F 3 "http://www.murata.com/~/media/webrenewal/support/library/catalog/products/emc/emifil/c31e.ashx?la=en-gb" V 9645 4745 50  0001 C CNN
+F 4 "W/FERRITE" H 9645 4745 50  0001 C CNN "EMI_FILTER_TYPE"
+F 5 "JOYSTICK" H 9645 4745 50  0001 C CNN "Optional"
 	1    9645 4745
 	-1   0    0    -1
@@
 F 2 "Raemixx500:EMI_Filter_Long" V 7455 4530 50  0001 C CNN
 F 3 "http://www.murata.com/~/media/webrenewal/support/library/catalog/products/emc/emifil/c31e.ashx?la=en-gb" V 7455 4530 50  0001 C CNN
+F 4 "W/FERRITE" H 7455 4530 50  0001 C CNN "EMI_FILTER_TYPE"
+F 5 "JOYSTICK" H 7455 4530 50  0001 C CNN "Optional"
 	1    7455 4530
 	1    0    0    -1
@@
 F 2 "Raemixx500:EMI_Filter_Long" V 7455 2300 50  0001 C CNN
 F 3 "http://www.murata.com/~/media/webrenewal/support/library/catalog/products/emc/emifil/c31e.ashx?la=en-gb" V 7455 2300 50  0001 C CNN
+F 4 "W/FERRITE" H 7455 2300 50  0001 C CNN "EMI_FILTER_TYPE"
+F 5 "JOYSTICK" H 7455 2300 50  0001 C CNN "Optional"
 	1    7455 2300
 	1    0    0    -1
@@
 F 2 "Raemixx500:EMI_Filter_Long" V 7090 4930 50  0001 C CNN
 F 3 "http://www.murata.com/~/media/webrenewal/support/library/catalog/products/emc/emifil/c31e.ashx?la=en-gb" V 7090 4930 50  0001 C CNN
+F 4 "W/FERRITE" H 7090 4930 50  0001 C CNN "EMI_FILTER_TYPE"
 	1    7090 4930
 	1    0    0    -1
@@
 F 2 "Raemixx500:EMI_Filter_Long" V 7090 2100 50  0001 C CNN
 F 3 "http://www.murata.com/~/media/webrenewal/support/library/catalog/products/emc/emifil/c31e.ashx?la=en-gb" V 7090 2100 50  0001 C CNN
+F 4 "W/FERRITE" H 7090 2100 50  0001 C CNN "EMI_FILTER_TYPE"
 	1    7090 2100
 	1    0    0    -1
