File: audio.sch (KiCad schematic (older format))
At the start: 94 parts, among them CN1 LEFT_JOY, CN2 RIGHT_JOY, CN3 RIGHT, CN4 LEFT, Q301 2N3906, Q321 MPF102, Q331 MPF102, U14 LF347, U15 74LS157, U3 PAULA, U38 MC1488

Commit message: Add part numbers for EMI filters Not the original filters, but what seem to be suitable replacements available today
Parts:
- E302, E303, E411, E412, E413, E414, E421, E422, E423, E424: Cost (none) -> 0.233; MFG Name (none) -> MURATA; MFG Part Num (none) -> DSS1NB32A682Q91A
- E305, E306: Cost (none) -> 0.233; MFG Name (none) -> MURATA; MFG Part Num (none) -> DSS1NB32A271Q91A
- E401, E408: Cost (none) -> 0.234; MFG Name (none) -> MURATA; MFG Part Num (none) -> DSS1NB32A151Q91A
- E415, E416, E417, E425, E426, E427, E441, E442, E443, E444: Cost (none) -> 0.233; MFG Name (none) -> MURATA; MFG Part Num (none) -> DSS1NB32A471Q91A
Changed lines of the file:
@@
 F 3 "http://www.murata.com/~/media/webrenewal/support/library/catalog/products/emc/emifil/c31e.ashx?la=en-gb" V 7090 2700 50  0001 C CNN
 F 4 "W/FERRITE" H 7090 2700 50  0001 C CNN "EMI_FILTER_TYPE"
+F 5 "0.233" H 7090 2700 50  0001 C CNN "Cost"
+F 6 "MURATA" H 7090 2700 50  0001 C CNN "MFG Name"
+F 7 "DSS1NB32A471Q91A" H 7090 2700 50  0001 C CNN "MFG Part Num"
 	1    7090 2700
 	1    0    0    -1
@@
 F 3 "http://www.murata.com/~/media/webrenewal/support/library/catalog/products/emc/emifil/c31e.ashx?la=en-gb" V 7580 2900 50  0001 C CNN
 F 4 "W/FERRITE" H 7580 2900 50  0001 C CNN "EMI_FILTER_TYPE"
+F 5 "0.233" H 7580 2900 50  0001 C CNN "Cost"
+F 6 "MURATA" H 7580 2900 50  0001 C CNN "MFG Name"
+F 7 "DSS1NB32A471Q91A" H 7580 2900 50  0001 C CNN "MFG Part Num"
 	1    7580 2900
 	1    0    0    -1
@@
 F 3 "http://www.murata.com/~/media/webrenewal/support/library/catalog/products/emc/emifil/c31e.ashx?la=en-gb" V 7090 4330 50  0001 C CNN
 F 4 "W/FERRITE" H 7090 4330 50  0001 C CNN "EMI_FILTER_TYPE"
+F 5 "0.233" H 7090 4330 50  0001 C CNN "Cost"
+F 6 "MURATA" H 7090 4330 50  0001 C CNN "MFG Name"
+F 7 "DSS1NB32A471Q91A" H 7090 4330 50  0001 C CNN "MFG Part Num"
 	1    7090 4330
 	1    0    0    -1
@@
 F 3 "http://www.murata.com/~/media/webrenewal/support/library/catalog/products/emc/emifil/c31e.ashx?la=en-gb" V 7580 5130 50  0001 C CNN
 F 4 "W/FERRITE" H 7580 5130 50  0001 C CNN "EMI_FILTER_TYPE"
+F 5 "0.233" H 7580 5130 50  0001 C CNN "Cost"
+F 6 "MURATA" H 7580 5130 50  0001 C CNN "MFG Name"
+F 7 "DSS1NB32A471Q91A" H 7580 5130 50  0001 C CNN "MFG Part Num"
 	1    7580 5130
 	1    0    0    -1
@@
 F 4 "W/FERRITE" H 9645 1685 50  0001 C CNN "EMI_FILTER_TYPE"
 F 5 "JOYSTICK" H 9645 1685 50  0001 C CNN "Optional"
+F 6 "0.233" H 9645 1685 50  0001 C CNN "Cost"
+F 7 "MURATA" H 9645 1685 50  0001 C CNN "MFG Name"
+F 8 "DSS1NB32A682Q91A" H 9645 1685 50  0001 C CNN "MFG Part Num"
 	1    9645 1685
 	-1   0    0    -1
@@
 F 4 "W/FERRITE" H 9645 2115 50  0001 C CNN "EMI_FILTER_TYPE"
 F 5 "JOYSTICK" H 9645 2115 50  0001 C CNN "Optional"
+F 6 "0.233" H 9645 2115 50  0001 C CNN "Cost"
+F 7 "MURATA" H 9645 2115 50  0001 C CNN "MFG Name"
+F 8 "DSS1NB32A682Q91A" H 9645 2115 50  0001 C CNN "MFG Part Num"
 	1    9645 2115
 	-1   0    0    -1
@@
 F 4 "W/FERRITE" H 9645 2515 50  0001 C CNN "EMI_FILTER_TYPE"
 F 5 "JOYSTICK" H 9645 2515 50  0001 C CNN "Optional"
+F 6 "0.233" H 9645 2515 50  0001 C CNN "Cost"
+F 7 "MURATA" H 9645 2515 50  0001 C CNN "MFG Name"
+F 8 "DSS1NB32A682Q91A" H 9645 2515 50  0001 C CNN "MFG Part Num"
 	1    9645 2515
 	-1   0    0    -1
@@
 F 4 "W/FERRITE" H 9645 3915 50  0001 C CNN "EMI_FILTER_TYPE"
 F 5 "JOYSTICK" H 9645 3915 50  0001 C CNN "Optional"
+F 6 "0.233" H 9645 3915 50  0001 C CNN "Cost"
+F 7 "MURATA" H 9645 3915 50  0001 C CNN "MFG Name"
+F 8 "DSS1NB32A682Q91A" H 9645 3915 50  0001 C CNN "MFG Part Num"
 	1    9645 3915
 	-1   0    0    -1
@@
 F 4 "W/FERRITE" H 9645 4345 50  0001 C CNN "EMI_FILTER_TYPE"
 F 5 "JOYSTICK" H 9645 4345 50  0001 C CNN "Optional"
+F 6 "0.233" H 9645 4345 50  0001 C CNN "Cost"
+F 7 "MURATA" H 9645 4345 50  0001 C CNN "MFG Name"
+F 8 "DSS1NB32A682Q91A" H 9645 4345 50  0001 C CNN "MFG Part Num"
 	1    9645 4345
 	-1   0    0    -1
@@
 F 4 "W/FERRITE" H 9645 5165 50  0001 C CNN "EMI_FILTER_TYPE"
 F 5 "JOYSTICK" H 9645 5165 50  0001 C CNN "Optional"
+F 6 "0.233" H 9645 5165 50  0001 C CNN "Cost"
+F 7 "MURATA" H 9645 5165 50  0001 C CNN "MFG Name"
+F 8 "DSS1NB32A682Q91A" H 9645 5165 50  0001 C CNN "MFG Part Num"
 	1    9645 5165
 	-1   0    0    -1
@@
 F 3 "http://www.murata.com/~/media/webrenewal/support/library/catalog/products/emc/emifil/c31e.ashx?la=en-gb" V 13420 2680 50  0001 C CNN
 F 4 "W/FERRITE" H 13420 2680 50  0001 C CNN "EMI_FILTER_TYPE"
+F 5 "0.233" H 13420 2680 50  0001 C CNN "Cost"
+F 6 "MURATA" H 13420 2680 50  0001 C CNN "MFG Name"
+F 7 "DSS1NB32A471Q91A" H 13420 2680 50  0001 C CNN "MFG Part Num"
 	1    13420 2680
 	1    0    0    -1
@@
 F 3 "http://www.murata.com/~/media/webrenewal/support/library/catalog/products/emc/emifil/c31e.ashx?la=en-gb" V 13420 3110 50  0001 C CNN
 F 4 "W/FERRITE" H 13420 3110 50  0001 C CNN "EMI_FILTER_TYPE"
+F 5 "0.233" H 13420 3110 50  0001 C CNN "Cost"
+F 6 "MURATA" H 13420 3110 50  0001 C CNN "MFG Name"
+F 7 "DSS1NB32A471Q91A" H 13420 3110 50  0001 C CNN "MFG Part Num"
 	1    13420 3110
 	1    0    0    -1
@@
 F 3 "http://www.murata.com/~/media/webrenewal/support/library/catalog/products/emc/emifil/c31e.ashx?la=en-gb" V 13420 3510 50  0001 C CNN
 F 4 "W/FERRITE" H 13420 3510 50  0001 C CNN "EMI_FILTER_TYPE"
+F 5 "0.233" H 13420 3510 50  0001 C CNN "Cost"
+F 6 "MURATA" H 13420 3510 50  0001 C CNN "MFG Name"
+F 7 "DSS1NB32A471Q91A" H 13420 3510 50  0001 C CNN "MFG Part Num"
 	1    13420 3510
 	1    0    0    -1
@@
 F 3 "http://www.murata.com/~/media/webrenewal/support/library/catalog/products/emc/emifil/c31e.ashx?la=en-gb" V 13420 3930 50  0001 C CNN
 F 4 "W/FERRITE" H 13420 3930 50  0001 C CNN "EMI_FILTER_TYPE"
+F 5 "0.233" H 13420 3930 50  0001 C CNN "Cost"
+F 6 "MURATA" H 13420 3930 50  0001 C CNN "MFG Name"
+F 7 "DSS1NB32A471Q91A" H 13420 3930 50  0001 C CNN "MFG Part Num"
 	1    13420 3930
 	1    0    0    -1
@@
 F 3 "http://www.murata.com/~/media/webrenewal/support/library/catalog/products/emc/emifil/c31e.ashx?la=en-gb" V 6310 7020 50  0001 C CNN
 F 4 "W/FERRITE" H 6310 7020 50  0001 C CNN "EMI_FILTER_TYPE"
+F 5 "0.233" H 6310 7020 50  0001 C CNN "Cost"
+F 6 "MURATA" H 6310 7020 50  0001 C CNN "MFG Name"
+F 7 "DSS1NB32A271Q91A" H 6310 7020 50  0001 C CNN "MFG Part Num"
 	1    6310 7020
 	1    0    0    -1
@@
 F 3 "http://www.murata.com/~/media/webrenewal/support/library/catalog/products/emc/emifil/c31e.ashx?la=en-gb" V 6310 8815 50  0001 C CNN
 F 4 "W/FERRITE" H 6310 8815 50  0001 C CNN "EMI_FILTER_TYPE"
+F 5 "0.233" H 6310 8815 50  0001 C CNN "Cost"
+F 6 "MURATA" H 6310 8815 50  0001 C CNN "MFG Name"
+F 7 "DSS1NB32A271Q91A" H 6310 8815 50  0001 C CNN "MFG Part Num"
 	1    6310 8815
 	1    0    0    -1
@@
 F 3 "http://www.murata.com/~/media/webrenewal/support/library/catalog/products/emc/emifil/c31e.ashx?la=en-gb" V 12020 9015 50  0001 C CNN
 F 4 "W/FERRITE" H 12020 9015 50  0001 C CNN "EMI_FILTER_TYPE"
+F 5 "0.233" H 12020 9015 50  0001 C CNN "Cost"
+F 6 "MURATA" H 12020 9015 50  0001 C CNN "MFG Name"
+F 7 "DSS1NB32A682Q91A" H 12020 9015 50  0001 C CNN "MFG Part Num"
 	1    12020 9015
 	1    0    0    -1
@@
 F 3 "http://www.murata.com/~/media/webrenewal/support/library/catalog/products/emc/emifil/c31e.ashx?la=en-gb" V 12020 7220 50  0001 C CNN
 F 4 "W/FERRITE" H 12020 7220 50  0001 C CNN "EMI_FILTER_TYPE"
+F 5 "0.233" H 12020 7220 50  0001 C CNN "Cost"
+F 6 "MURATA" H 12020 7220 50  0001 C CNN "MFG Name"
+F 7 "DSS1NB32A682Q91A" H 12020 7220 50  0001 C CNN "MFG Part Num"
 	1    12020 7220
 	1    0    0    -1
@@
 F 4 "W/FERRITE" H 9645 2935 50  0001 C CNN "EMI_FILTER_TYPE"
 F 5 "JOYSTICK" H 9645 2935 50  0001 C CNN "Optional"
+F 6 "0.233" H 9645 2935 50  0001 C CNN "Cost"
+F 7 "MURATA" H 9645 2935 50  0001 C CNN "MFG Name"
+F 8 "DSS1NB32A682Q91A" H 9645 2935 50  0001 C CNN "MFG Part Num"
 	1    9645 2935
 	-1   0    0    -1
@@
 F 4 "W/FERRITE" H 9645 4745 50  0001 C CNN "EMI_FILTER_TYPE"
 F 5 "JOYSTICK" H 9645 4745 50  0001 C CNN "Optional"
+F 6 "0.233" H 9645 4745 50  0001 C CNN "Cost"
+F 7 "MURATA" H 9645 4745 50  0001 C CNN "MFG Name"
+F 8 "DSS1NB32A682Q91A" H 9645 4745 50  0001 C CNN "MFG Part Num"
 	1    9645 4745
 	-1   0    0    -1
@@
 F 4 "W/FERRITE" H 7455 4530 50  0001 C CNN "EMI_FILTER_TYPE"
 F 5 "JOYSTICK" H 7455 4530 50  0001 C CNN "Optional"
+F 6 "0.234" H 7455 4530 50  0001 C CNN "Cost"
+F 7 "MURATA" H 7455 4530 50  0001 C CNN "MFG Name"
+F 8 "DSS1NB32A151Q91A" H 7455 4530 50  0001 C CNN "MFG Part Num"
 	1    7455 4530
 	1    0    0    -1
@@
 F 4 "W/FERRITE" H 7455 2300 50  0001 C CNN "EMI_FILTER_TYPE"
 F 5 "JOYSTICK" H 7455 2300 50  0001 C CNN "Optional"
+F 6 "0.234" H 7455 2300 50  0001 C CNN "Cost"
+F 7 "MURATA" H 7455 2300 50  0001 C CNN "MFG Name"
+F 8 "DSS1NB32A151Q91A" H 7455 2300 50  0001 C CNN "MFG Part Num"
 	1    7455 2300
 	1    0    0    -1
@@
 F 3 "http://www.murata.com/~/media/webrenewal/support/library/catalog/products/emc/emifil/c31e.ashx?la=en-gb" V 7090 4930 50  0001 C CNN
 F 4 "W/FERRITE" H 7090 4930 50  0001 C CNN "EMI_FILTER_TYPE"
+F 5 "0.233" H 7090 4930 50  0001 C CNN "Cost"
+F 6 "MURATA" H 7090 4930 50  0001 C CNN "MFG Name"
+F 7 "DSS1NB32A471Q91A" H 7090 4930 50  0001 C CNN "MFG Part Num"
 	1    7090 4930
 	1    0    0    -1
@@
 F 3 "http://www.murata.com/~/media/webrenewal/support/library/catalog/products/emc/emifil/c31e.ashx?la=en-gb" V 7090 2100 50  0001 C CNN
 F 4 "W/FERRITE" H 7090 2100 50  0001 C CNN "EMI_FILTER_TYPE"
+F 5 "0.233" H 7090 2100 50  0001 C CNN "Cost"
+F 6 "MURATA" H 7090 2100 50  0001 C CNN "MFG Name"
+F 7 "DSS1NB32A471Q91A" H 7090 2100 50  0001 C CNN "MFG Part Num"
 	1    7090 2100
 	1    0    0    -1

Commit message: Add EMI filter 3D models, add logo, re-add Rock Lobster (closes #15) Thanks to Szabó Zoltán and Workshopshed!
Parts:
- E401, E408: MFG Part Num DSS1NB32A151Q91A -> DSS1NB32A103Q91A
Changed lines of the file:
@@
 F 6 "0.234" H 7455 4530 50  0001 C CNN "Cost"
 F 7 "MURATA" H 7455 4530 50  0001 C CNN "MFG Name"
-F 8 "DSS1NB32A151Q91A" H 7455 4530 50  0001 C CNN "MFG Part Num"
+F 8 "DSS1NB32A103Q91A" H 7455 4530 50  0001 C CNN "MFG Part Num"
 	1    7455 4530
 	1    0    0    -1
@@
 F 6 "0.234" H 7455 2300 50  0001 C CNN "Cost"
 F 7 "MURATA" H 7455 2300 50  0001 C CNN "MFG Name"
-F 8 "DSS1NB32A151Q91A" H 7455 2300 50  0001 C CNN "MFG Part Num"
+F 8 "DSS1NB32A103Q91A" H 7455 2300 50  0001 C CNN "MFG Part Num"
 	1    7455 2300
 	1    0    0    -1

Commit message: (Try to) Identify the minimum set of required components
Parts:
- C3, C305, C306, C307: Required (none) -> R
- FB802, R303, R304, R309, U3: Required (none) -> Y
Changed lines of the file:
@@
 F 3 "DOCUMENTATION" H 3125 5655 50  0001 C CNN
 F 4 "CUSTOM" H 3125 5655 50  0001 C CNN "Optional"
+F 5 "Y" H 3125 5655 50  0001 C CNN "Required"
 	1    3125 5655
 	1    0    0    -1
@@
 F 3 "~" H 4330 8070 50  0001 C CNN
 F 4 "FERRITE" H 4330 8070 50  0001 C CNN "EMI_FILTER_TYPE"
+F 5 "Y" H 4330 8070 50  0001 C CNN "Required"
 	1    4330 8070
 	1    0    0    -1
@@
 F 3 "DOCUMENTATION" H 1125 2160 50  0001 C CNN
 F 4 "CUSTOM" H 1125 2160 50  0001 C CNN "Optional"
+F 5 "Y" H 1125 2160 50  0001 C CNN "Required"
 	2    1125 2160
 	1    0    0    -1
@@
 F 2 "Resistor_THT:R_Axial_DIN0309_L9.0mm_D3.2mm_P15.24mm_Horizontal" V 1055 1275 50  0001 C CNN
 F 3 "~" H 1125 1275 50  0001 C CNN
+F 4 "Y" H 1125 1275 50  0001 C CNN "Required"
 	1    1125 1275
 	1    0    0    -1
@@
 F 5 "C412C334M5U5TA" H 1825 2115 50  0001 C CNN "MFG Part Num"
 F 6 "0.078" H 1825 2115 50  0001 C CNN "Cost"
+F 7 "R" H 1825 2115 50  0001 C CNN "Required"
 	1    1825 2115
 	1    0    0    -1
@@
 F 2 "Raemixx500:R_Axial_DIN0309_L9.0mm_D3.2mm_P12.70mm_Horizontal" V 2625 1515 50  0001 C CNN
 F 3 "~" H 2695 1515 50  0001 C CNN
+F 4 "Y" H 2695 1515 50  0001 C CNN "Required"
 	1    2695 1515
 	0    1    1    0
@@
 F 5 "PANASONIC" H 2245 2115 50  0001 C CNN "MFG Name"
 F 6 "EEUFR1C102" H 2245 2115 50  0001 C CNN "MFG Part Num"
+F 7 "R" H 2245 2115 50  0001 C CNN "Required"
 	1    2245 2115
 	1    0    0    -1
@@
 F 2 "Raemixx500:R_Axial_DIN0309_L9.0mm_D3.2mm_P12.70mm_Horizontal" V 3075 2115 50  0001 C CNN
 F 3 "~" H 3145 2115 50  0001 C CNN
+F 4 "Y" H 3145 2115 50  0001 C CNN "Required"
 	1    3145 2115
 	-1   0    0    1
@@
 F 5 "C412C334M5U5TA" H 3845 2115 50  0001 C CNN "MFG Part Num"
 F 6 "0.078" H 3845 2115 50  0001 C CNN "Cost"
+F 7 "R" H 3845 2115 50  0001 C CNN "Required"
 	1    3845 2115
 	1    0    0    -1
@@
 F 5 "PANASONIC" H 4265 2115 50  0001 C CNN "MFG Name"
 F 6 "EEUFR1H100" H 4265 2115 50  0001 C CNN "MFG Part Num"
+F 7 "R" H 4265 2115 50  0001 C CNN "Required"
 	1    4265 2115
 	1    0    0    -1

Commit message: Rename "Optional" Field to "Section"
Parts:
- CN1, CN2, E401, E408, E411, E412, E413, E414, E421, E422, E423, E424, U15: Optional JOYSTICK -> (none); Section (none) -> JOYSTICK
- CN3, CN4, U14: Optional AUDIO -> (none); Section (none) -> AUDIO
- JP10A1, JP10B1, JP8: Optional JMP -> (none); Section (none) -> JMP
- U3: Optional CUSTOM -> (none); Section (none) -> CUSTOM
- U38: Optional SERIAL -> (none); Section (none) -> SERIAL
Changed lines of the file:
@@
 F 2 "Package_DIP:DIP-48_W15.24mm_Socket_LongPads" H 3125 5655 50  0001 C CNN
 F 3 "DOCUMENTATION" H 3125 5655 50  0001 C CNN
-F 4 "CUSTOM" H 3125 5655 50  0001 C CNN "Optional"
+F 4 "CUSTOM" H 3125 5655 50  0001 C CNN "Section"
 F 5 "Y" H 3125 5655 50  0001 C CNN "Required"
 	1    3125 5655
@@
 F 2 "Raemixx500:DB_9M" H 8775 2300 50  0001 C CNN
 F 3 " ~" H 8775 2300 50  0001 C CNN
-F 4 "JOYSTICK" H 8775 2300 50  0001 C CNN "Optional"
+F 4 "JOYSTICK" H 8775 2300 50  0001 C CNN "Section"
 	1    8775 2300
 	-1   0    0    1
@@
 F 4 "SKIP" H 5645 2440 50  0001 C CNN "MFG Name"
 F 5 "SKIP" H 5645 2440 50  0001 C CNN "MFG Part Num"
-F 6 "JMP" H 5645 2440 50  0001 C CNN "Optional"
+F 6 "JMP" H 5645 2440 50  0001 C CNN "Section"
 	1    5645 2440
 	0    1    1    0
@@
 F 2 "Raemixx500:DB_9M" H 8775 4530 50  0001 C CNN
 F 3 " ~" H 8775 4530 50  0001 C CNN
-F 4 "JOYSTICK" H 8775 4530 50  0001 C CNN "Optional"
+F 4 "JOYSTICK" H 8775 4530 50  0001 C CNN "Section"
 	1    8775 4530
 	-1   0    0    1
@@
 F 3 "http://www.murata.com/~/media/webrenewal/support/library/catalog/products/emc/emifil/c31e.ashx?la=en-gb" V 9645 1685 50  0001 C CNN
 F 4 "W/FERRITE" H 9645 1685 50  0001 C CNN "EMI_FILTER_TYPE"
-F 5 "JOYSTICK" H 9645 1685 50  0001 C CNN "Optional"
+F 5 "JOYSTICK" H 9645 1685 50  0001 C CNN "Section"
 F 6 "0.233" H 9645 1685 50  0001 C CNN "Cost"
 F 7 "MURATA" H 9645 1685 50  0001 C CNN "MFG Name"
@@
 F 3 "http://www.murata.com/~/media/webrenewal/support/library/catalog/products/emc/emifil/c31e.ashx?la=en-gb" V 9645 2115 50  0001 C CNN
 F 4 "W/FERRITE" H 9645 2115 50  0001 C CNN "EMI_FILTER_TYPE"
-F 5 "JOYSTICK" H 9645 2115 50  0001 C CNN "Optional"
+F 5 "JOYSTICK" H 9645 2115 50  0001 C CNN "Section"
 F 6 "0.233" H 9645 2115 50  0001 C CNN "Cost"
 F 7 "MURATA" H 9645 2115 50  0001 C CNN "MFG Name"
@@
 F 3 "http://www.murata.com/~/media/webrenewal/support/library/catalog/products/emc/emifil/c31e.ashx?la=en-gb" V 9645 2515 50  0001 C CNN
 F 4 "W/FERRITE" H 9645 2515 50  0001 C CNN "EMI_FILTER_TYPE"
-F 5 "JOYSTICK" H 9645 2515 50  0001 C CNN "Optional"
+F 5 "JOYSTICK" H 9645 2515 50  0001 C CNN "Section"
 F 6 "0.233" H 9645 2515 50  0001 C CNN "Cost"
 F 7 "MURATA" H 9645 2515 50  0001 C CNN "MFG Name"
@@
 F 2 "Package_DIP:DIP-16_W7.62mm_Socket_LongPads" H 12455 3375 50  0001 C CNN
 F 3 "http://www.ti.com/lit/gpn/sn74LS157" H 12455 3375 50  0001 C CNN
-F 4 "JOYSTICK" H 12455 3375 50  0001 C CNN "Optional"
+F 4 "JOYSTICK" H 12455 3375 50  0001 C CNN "Section"
 F 5 "0.236" H 12455 3375 50  0001 C CNN "Cost"
 F 6 "TI" H 12455 3375 50  0001 C CNN "MFG Name"
@@
 F 3 "http://www.murata.com/~/media/webrenewal/support/library/catalog/products/emc/emifil/c31e.ashx?la=en-gb" V 9645 3915 50  0001 C CNN
 F 4 "W/FERRITE" H 9645 3915 50  0001 C CNN "EMI_FILTER_TYPE"
-F 5 "JOYSTICK" H 9645 3915 50  0001 C CNN "Optional"
+F 5 "JOYSTICK" H 9645 3915 50  0001 C CNN "Section"
 F 6 "0.233" H 9645 3915 50  0001 C CNN "Cost"
 F 7 "MURATA" H 9645 3915 50  0001 C CNN "MFG Name"
@@
 F 3 "http://www.murata.com/~/media/webrenewal/support/library/catalog/products/emc/emifil/c31e.ashx?la=en-gb" V 9645 4345 50  0001 C CNN
 F 4 "W/FERRITE" H 9645 4345 50  0001 C CNN "EMI_FILTER_TYPE"
-F 5 "JOYSTICK" H 9645 4345 50  0001 C CNN "Optional"
+F 5 "JOYSTICK" H 9645 4345 50  0001 C CNN "Section"
 F 6 "0.233" H 9645 4345 50  0001 C CNN "Cost"
 F 7 "MURATA" H 9645 4345 50  0001 C CNN "MFG Name"
@@
 F 3 "http://www.murata.com/~/media/webrenewal/support/library/catalog/products/emc/emifil/c31e.ashx?la=en-gb" V 9645 5165 50  0001 C CNN
 F 4 "W/FERRITE" H 9645 5165 50  0001 C CNN "EMI_FILTER_TYPE"
-F 5 "JOYSTICK" H 9645 5165 50  0001 C CNN "Optional"
+F 5 "JOYSTICK" H 9645 5165 50  0001 C CNN "Section"
 F 6 "0.233" H 9645 5165 50  0001 C CNN "Cost"
 F 7 "MURATA" H 9645 5165 50  0001 C CNN "MFG Name"
@@
 F 2 "Package_DIP:DIP-14_W7.62mm_Socket_LongPads" H 9515 9015 50  0001 C CNN
 F 3 "http://www.ti.com/lit/ds/symlink/tl081.pdf" H 9615 9115 50  0001 C CNN
-F 4 "AUDIO" H 9565 8915 50  0001 C CNN "Optional"
+F 4 "AUDIO" H 9565 8915 50  0001 C CNN "Section"
 F 5 "0.58" H 9565 8915 50  0001 C CNN "Cost"
 F 6 "TI" H 9565 8915 50  0001 C CNN "MFG Name"
@@
 F 2 "Package_DIP:DIP-14_W7.62mm_Socket_LongPads" H 9515 7220 50  0001 C CNN
 F 3 "http://www.ti.com/lit/ds/symlink/tl081.pdf" H 9615 7320 50  0001 C CNN
-F 4 "AUDIO" H 9565 7120 50  0001 C CNN "Optional"
+F 4 "AUDIO" H 9565 7120 50  0001 C CNN "Section"
 F 5 "0.58" H 9565 7120 50  0001 C CNN "Cost"
 F 6 "TI" H 9565 7120 50  0001 C CNN "MFG Name"
@@
 F 2 "Package_DIP:DIP-14_W7.62mm_Socket_LongPads" H 7565 7120 50  0001 C CNN
 F 3 "http://www.ti.com/lit/ds/symlink/tl081.pdf" H 7665 7220 50  0001 C CNN
-F 4 "AUDIO" H 7615 7020 50  0001 C CNN "Optional"
+F 4 "AUDIO" H 7615 7020 50  0001 C CNN "Section"
 F 5 "0.58" H 7615 7020 50  0001 C CNN "Cost"
 F 6 "TI" H 7615 7020 50  0001 C CNN "MFG Name"
@@
 F 2 "Package_DIP:DIP-14_W7.62mm_Socket_LongPads" H 7565 8915 50  0001 C CNN
 F 3 "http://www.ti.com/lit/ds/symlink/tl081.pdf" H 7665 9015 50  0001 C CNN
-F 4 "AUDIO" H 7615 8815 50  0001 C CNN "Optional"
+F 4 "AUDIO" H 7615 8815 50  0001 C CNN "Section"
 F 5 "0.58" H 7615 8815 50  0001 C CNN "Cost"
 F 6 "TI" H 7615 8815 50  0001 C CNN "MFG Name"
@@
 F 2 "Package_DIP:DIP-14_W7.62mm_Socket_LongPads" H 3835 9285 50  0001 C CNN
 F 3 "DOCUMENTATION" H 3835 9285 50  0001 C CNN
-F 4 "SERIAL" H 3835 9285 50  0001 C CNN "Optional"
+F 4 "SERIAL" H 3835 9285 50  0001 C CNN "Section"
 F 5 "0.615" H 3835 9285 50  0001 C CNN "Cost"
 F 6 "TI" H 3835 9285 50  0001 C CNN "MFG Name"
@@
 F 4 "SKIP" H 11260 8440 50  0001 C CNN "MFG Name"
 F 5 "SKIP" H 11260 8440 50  0001 C CNN "MFG Part Num"
-F 6 "JMP" H 11260 8440 50  0001 C CNN "Optional"
+F 6 "JMP" H 11260 8440 50  0001 C CNN "Section"
 	1    11260 8440
 	1    0    0    -1
@@
 F 4 "SKIP" H 6150 6455 50  0001 C CNN "MFG Name"
 F 5 "SKIP" H 6150 6455 50  0001 C CNN "MFG Part Num"
-F 6 "JMP" H 6150 6455 50  0001 C CNN "Optional"
+F 6 "JMP" H 6150 6455 50  0001 C CNN "Section"
 	1    6150 6455
 	1    0    0    -1
@@
 F 2 "Package_DIP:DIP-48_W15.24mm_Socket_LongPads" H 1125 2160 50  0001 C CNN
 F 3 "DOCUMENTATION" H 1125 2160 50  0001 C CNN
-F 4 "CUSTOM" H 1125 2160 50  0001 C CNN "Optional"
+F 4 "CUSTOM" H 1125 2160 50  0001 C CNN "Section"
 F 5 "Y" H 1125 2160 50  0001 C CNN "Required"
 	2    1125 2160
@@
 F 2 "Package_DIP:DIP-14_W7.62mm_Socket_LongPads" H 1240 9805 50  0001 C CNN
 F 3 "http://www.ti.com/lit/ds/symlink/tl081.pdf" H 1340 9905 50  0001 C CNN
-F 4 "AUDIO" H 1290 9705 50  0001 C CNN "Optional"
+F 4 "AUDIO" H 1290 9705 50  0001 C CNN "Section"
 F 5 "0.58" H 1290 9705 50  0001 C CNN "Cost"
 F 6 "TI" H 1290 9705 50  0001 C CNN "MFG Name"
@@
 F 2 "Package_DIP:DIP-16_W7.62mm_Socket_LongPads" H 14900 3345 50  0001 C CNN
 F 3 "http://www.ti.com/lit/gpn/sn74LS157" H 14900 3345 50  0001 C CNN
-F 4 "JOYSTICK" H 14900 3345 50  0001 C CNN "Optional"
+F 4 "JOYSTICK" H 14900 3345 50  0001 C CNN "Section"
 F 5 "0.236" H 14900 3345 50  0001 C CNN "Cost"
 F 6 "TI" H 14900 3345 50  0001 C CNN "MFG Name"
@@
 F 3 "http://www.murata.com/~/media/webrenewal/support/library/catalog/products/emc/emifil/c31e.ashx?la=en-gb" V 9645 2935 50  0001 C CNN
 F 4 "W/FERRITE" H 9645 2935 50  0001 C CNN "EMI_FILTER_TYPE"
-F 5 "JOYSTICK" H 9645 2935 50  0001 C CNN "Optional"
+F 5 "JOYSTICK" H 9645 2935 50  0001 C CNN "Section"
 F 6 "0.233" H 9645 2935 50  0001 C CNN "Cost"
 F 7 "MURATA" H 9645 2935 50  0001 C CNN "MFG Name"
@@
 F 3 "http://www.murata.com/~/media/webrenewal/support/library/catalog/products/emc/emifil/c31e.ashx?la=en-gb" V 9645 4745 50  0001 C CNN
 F 4 "W/FERRITE" H 9645 4745 50  0001 C CNN "EMI_FILTER_TYPE"
-F 5 "JOYSTICK" H 9645 4745 50  0001 C CNN "Optional"
+F 5 "JOYSTICK" H 9645 4745 50  0001 C CNN "Section"
 F 6 "0.233" H 9645 4745 50  0001 C CNN "Cost"
 F 7 "MURATA" H 9645 4745 50  0001 C CNN "MFG Name"
@@
 F 3 "http://www.murata.com/~/media/webrenewal/support/library/catalog/products/emc/emifil/c31e.ashx?la=en-gb" V 7455 4530 50  0001 C CNN
 F 4 "W/FERRITE" H 7455 4530 50  0001 C CNN "EMI_FILTER_TYPE"
-F 5 "JOYSTICK" H 7455 4530 50  0001 C CNN "Optional"
+F 5 "JOYSTICK" H 7455 4530 50  0001 C CNN "Section"
 F 6 "0.234" H 7455 4530 50  0001 C CNN "Cost"
 F 7 "MURATA" H 7455 4530 50  0001 C CNN "MFG Name"
@@
 F 3 "http://www.murata.com/~/media/webrenewal/support/library/catalog/products/emc/emifil/c31e.ashx?la=en-gb" V 7455 2300 50  0001 C CNN
 F 4 "W/FERRITE" H 7455 2300 50  0001 C CNN "EMI_FILTER_TYPE"
-F 5 "JOYSTICK" H 7455 2300 50  0001 C CNN "Optional"
+F 5 "JOYSTICK" H 7455 2300 50  0001 C CNN "Section"
 F 6 "0.234" H 7455 2300 50  0001 C CNN "Cost"
 F 7 "MURATA" H 7455 2300 50  0001 C CNN "MFG Name"
@@
 F 5 "13mm" H 12965 7320 50  0001 L BNN "Field5"
 F 6 "Manufacturer Recommendations" H 12965 7320 50  0001 L BNN "Field6"
-F 7 "AUDIO" H 12965 7320 50  0001 C CNN "Optional"
+F 7 "AUDIO" H 12965 7320 50  0001 C CNN "Section"
 	1    12965 7320
 	-1   0    0    -1
@@
 F 5 "13mm" H 12965 9115 50  0001 L BNN "Field5"
 F 6 "Manufacturer Recommendations" H 12965 9115 50  0001 L BNN "Field6"
-F 7 "AUDIO" H 12965 9115 50  0001 C CNN "Optional"
+F 7 "AUDIO" H 12965 9115 50  0001 C CNN "Section"
 	1    12965 9115
 	-1   0    0    -1
