File: clockdist.sch (KiCad schematic (older format))
At the start: 16 parts, among them U33 74LS258

Commit message: Begin adding part numbers
Parts:
- C33: Cost (none) -> 0.071; MFG Name (none) -> KEMET; MFG Part Num (none) -> C410C103K1H5TAAUTO
- U33: Optional (none) -> CLOCK
Changed lines of the file:
@@
 F 2 "Package_DIP:DIP-16_W7.62mm_Socket_LongPads" H 3640 2550 50  0001 C CNN
 F 3 "http://www.ti.com/lit/gpn/sn74LS258" H 3640 2550 50  0001 C CNN
+F 4 "CLOCK" H 3640 2550 50  0001 C CNN "Optional"
 	1    3640 2550
 	1    0    0    -1
@@
 F 2 "Package_DIP:DIP-16_W7.62mm_Socket_LongPads" H 6740 1650 50  0001 C CNN
 F 3 "http://www.ti.com/lit/gpn/sn74LS258" H 6740 1650 50  0001 C CNN
+F 4 "CLOCK" H 3640 3950 50  0001 C CNN "Optional"
 	2    3640 3950
 	1    0    0    -1
@@
 F 2 "Package_DIP:DIP-16_W7.62mm_Socket_LongPads" H 6740 950 50  0001 C CNN
 F 3 "http://www.ti.com/lit/gpn/sn74LS258" H 6740 950 50  0001 C CNN
+F 4 "CLOCK" H 3640 3250 50  0001 C CNN "Optional"
 	3    3640 3250
 	1    0    0    -1
@@
 F 2 "Package_DIP:DIP-16_W7.62mm_Socket_LongPads" H 12890 1470 50  0001 C CNN
 F 3 "http://www.ti.com/lit/gpn/sn74LS258" H 12890 1470 50  0001 C CNN
+F 4 "CLOCK" H 9790 3770 50  0001 C CNN "Optional"
 	5    9790 3770
 	1    0    0    -1
@@
 F 2 "Raemixx500:C_Axial_L6.3mm_D2.5mm_P10.16mm" H 10228 3720 50  0001 C CNN
 F 3 "~" H 10190 3870 50  0001 C CNN
+F 4 "KEMET" H 10190 3870 50  0001 C CNN "MFG Name"
+F 5 "C410C103K1H5TAAUTO" H 10190 3870 50  0001 C CNN "MFG Part Num"
+F 6 "0.071" H 10190 3870 50  0001 C CNN "Cost"
 	1    10190 3870
 	1    0    0    -1

Commit message: More part numbers
Parts:
- C33, E102, E103, E104, E105, E106, E107, E108, E109, E407, E791, E792, E793, E794, RP103: Optional (none) -> CLOCK
- U33: MFG Name (none) -> N/A
Changed lines of the file:
@@
 F 3 "http://www.ti.com/lit/gpn/sn74LS258" H 3640 2550 50  0001 C CNN
 F 4 "CLOCK" H 3640 2550 50  0001 C CNN "Optional"
+F 5 "N/A" H 3640 2550 50  0001 C CNN "MFG Name"
 	1    3640 2550
 	1    0    0    -1
@@
 F 3 "http://www.ti.com/lit/gpn/sn74LS258" H 6740 1650 50  0001 C CNN
 F 4 "CLOCK" H 3640 3950 50  0001 C CNN "Optional"
+F 5 "N/A" H 3640 3950 50  0001 C CNN "MFG Name"
 	2    3640 3950
 	1    0    0    -1
@@
 F 3 "http://www.ti.com/lit/gpn/sn74LS258" H 6740 950 50  0001 C CNN
 F 4 "CLOCK" H 3640 3250 50  0001 C CNN "Optional"
+F 5 "N/A" H 3640 3250 50  0001 C CNN "MFG Name"
 	3    3640 3250
 	1    0    0    -1
@@
 F 2 "Resistor_THT:R_Array_SIP10" V 5615 3250 50  0001 C CNN
 F 3 "~" H 5240 3250 50  0001 C CNN
+F 4 "CLOCK" H 5240 3250 50  0001 C CNN "Optional"
 	1    5240 3250
 	0    1    1    0
@@
 F 3 "http://www.ti.com/lit/gpn/sn74LS258" H 12890 1470 50  0001 C CNN
 F 4 "CLOCK" H 9790 3770 50  0001 C CNN "Optional"
+F 5 "N/A" H 9790 3770 50  0001 C CNN "MFG Name"
 	5    9790 3770
 	1    0    0    -1
@@
 F 5 "C410C103K1H5TAAUTO" H 10190 3870 50  0001 C CNN "MFG Part Num"
 F 6 "0.071" H 10190 3870 50  0001 C CNN "Cost"
+F 7 "CLOCK" H 10190 3870 50  0001 C CNN "Optional"
 	1    10190 3870
 	1    0    0    -1
@@
 F 2 "Raemixx500:C_Axial_L6.3mm_D2.5mm_P10.16mm" H 6148 4620 50  0001 C CNN
 F 3 "~" H 6110 4770 50  0001 C CNN
+F 4 "CLOCK" H 6110 4770 50  0001 C CNN "Optional"
 	1    6110 4770
 	1    0    0    -1
@@
 F 2 "Raemixx500:C_Axial_L6.3mm_D2.5mm_P10.16mm" H 6588 4630 50  0001 C CNN
 F 3 "~" H 6550 4780 50  0001 C CNN
+F 4 "CLOCK" H 6550 4780 50  0001 C CNN "Optional"
 	1    6550 4780
 	1    0    0    -1
@@
 F 2 "Raemixx500:C_Axial_L6.3mm_D2.5mm_P10.16mm" H 7028 4630 50  0001 C CNN
 F 3 "~" H 6990 4780 50  0001 C CNN
+F 4 "CLOCK" H 6990 4780 50  0001 C CNN "Optional"
 	1    6990 4780
 	1    0    0    -1
@@
 F 2 "Raemixx500:C_Axial_L6.3mm_D2.5mm_P10.16mm" H 7468 4640 50  0001 C CNN
 F 3 "~" H 7430 4790 50  0001 C CNN
+F 4 "CLOCK" H 7430 4790 50  0001 C CNN "Optional"
 	1    7430 4790
 	1    0    0    -1
@@
 F 2 "Raemixx500:C_Axial_L9.0mm_D3.2mm_P12.70mm" H 7908 4640 50  0001 C CNN
 F 3 "~" H 7870 4790 50  0001 C CNN
+F 4 "CLOCK" H 7870 4790 50  0001 C CNN "Optional"
 	1    7870 4790
 	1    0    0    -1
@@
 F 2 "Raemixx500:C_Axial_L9.0mm_D3.2mm_P12.70mm" H 2038 4610 50  0001 C CNN
 F 3 "~" H 2000 4760 50  0001 C CNN
+F 4 "CLOCK" H 2000 4760 50  0001 C CNN "Optional"
 	1    2000 4760
 	1    0    0    -1
@@
 F 2 "Raemixx500:C_Axial_L9.0mm_D3.2mm_P12.70mm" H 2478 4620 50  0001 C CNN
 F 3 "~" H 2440 4770 50  0001 C CNN
+F 4 "CLOCK" H 2440 4770 50  0001 C CNN "Optional"
 	1    2440 4770
 	1    0    0    -1
@@
 F 2 "Raemixx500:C_Axial_L9.0mm_D3.2mm_P12.70mm" H 2918 4620 50  0001 C CNN
 F 3 "~" H 2880 4770 50  0001 C CNN
+F 4 "CLOCK" H 2880 4770 50  0001 C CNN "Optional"
 	1    2880 4770
 	1    0    0    -1
@@
 F 2 "Raemixx500:C_Axial_L6.3mm_D2.5mm_P10.16mm" H 2478 6640 50  0001 C CNN
 F 3 "~" H 2440 6790 50  0001 C CNN
+F 4 "CLOCK" H 2440 6790 50  0001 C CNN "Optional"
 	1    2440 6790
 	1    0    0    -1
@@
 F 2 "Raemixx500:C_Axial_L9.0mm_D3.2mm_P12.70mm" H 2918 6650 50  0001 C CNN
 F 3 "~" H 2880 6800 50  0001 C CNN
+F 4 "CLOCK" H 2880 6800 50  0001 C CNN "Optional"
 	1    2880 6800
 	1    0    0    -1
@@
 F 2 "Raemixx500:EMI_Filter_Short" V 9690 2870 50  0001 C CNN
 F 3 "http://www.murata.com/~/media/webrenewal/support/library/catalog/products/emc/emifil/c31e.ashx?la=en-gb" V 9690 2870 50  0001 C CNN
+F 4 "CLOCK" H 9690 2870 50  0001 C CNN "Optional"
 	1    9690 2870
 	0    1    1    0
@@
 F 2 "Raemixx500:EMI_Filter_Long" V 5390 4050 50  0001 C CNN
 F 3 "http://www.murata.com/~/media/webrenewal/support/library/catalog/products/emc/emifil/c31e.ashx?la=en-gb" V 5390 4050 50  0001 C CNN
+F 4 "CLOCK" H 5390 4050 50  0001 C CNN "Optional"
 	1    5390 4050
 	1    0    0    -1
@@
 F 2 "Raemixx500:EMI_Filter_Long" V 5390 4450 50  0001 C CNN
 F 3 "http://www.murata.com/~/media/webrenewal/support/library/catalog/products/emc/emifil/c31e.ashx?la=en-gb" V 5390 4450 50  0001 C CNN
+F 4 "CLOCK" H 5390 4450 50  0001 C CNN "Optional"
 	1    5390 4450
 	1    0    0    -1

Commit message: Add EMI filter types
Parts:
- E102, E103, E106, E107, E108, E109, E791, E792, E793, E794: EMI_FILTER_TYPE (none) -> C
- E104, E105: EMI_FILTER_TYPE (none) -> R
- E407: EMI_FILTER_TYPE (none) -> W/FERRITE
Changed lines of the file:
@@
 F 3 "~" H 6110 4770 50  0001 C CNN
 F 4 "CLOCK" H 6110 4770 50  0001 C CNN "Optional"
+F 5 "C" H 6110 4770 50  0001 C CNN "EMI_FILTER_TYPE"
 	1    6110 4770
 	1    0    0    -1
@@
 F 3 "~" H 6550 4780 50  0001 C CNN
 F 4 "CLOCK" H 6550 4780 50  0001 C CNN "Optional"
+F 5 "C" H 6550 4780 50  0001 C CNN "EMI_FILTER_TYPE"
 	1    6550 4780
 	1    0    0    -1
@@
 F 3 "~" H 6990 4780 50  0001 C CNN
 F 4 "CLOCK" H 6990 4780 50  0001 C CNN "Optional"
+F 5 "C" H 6990 4780 50  0001 C CNN "EMI_FILTER_TYPE"
 	1    6990 4780
 	1    0    0    -1
@@
 F 3 "~" H 7430 4790 50  0001 C CNN
 F 4 "CLOCK" H 7430 4790 50  0001 C CNN "Optional"
+F 5 "C" H 7430 4790 50  0001 C CNN "EMI_FILTER_TYPE"
 	1    7430 4790
 	1    0    0    -1
@@
 F 3 "~" H 7870 4790 50  0001 C CNN
 F 4 "CLOCK" H 7870 4790 50  0001 C CNN "Optional"
+F 5 "C" H 7870 4790 50  0001 C CNN "EMI_FILTER_TYPE"
 	1    7870 4790
 	1    0    0    -1
@@
 F 3 "~" H 2000 4760 50  0001 C CNN
 F 4 "CLOCK" H 2000 4760 50  0001 C CNN "Optional"
+F 5 "C" H 2000 4760 50  0001 C CNN "EMI_FILTER_TYPE"
 	1    2000 4760
 	1    0    0    -1
@@
 F 3 "~" H 2440 4770 50  0001 C CNN
 F 4 "CLOCK" H 2440 4770 50  0001 C CNN "Optional"
+F 5 "C" H 2440 4770 50  0001 C CNN "EMI_FILTER_TYPE"
 	1    2440 4770
 	1    0    0    -1
@@
 F 3 "~" H 2880 4770 50  0001 C CNN
 F 4 "CLOCK" H 2880 4770 50  0001 C CNN "Optional"
+F 5 "C" H 2880 4770 50  0001 C CNN "EMI_FILTER_TYPE"
 	1    2880 4770
 	1    0    0    -1
@@
 F 3 "~" H 2440 6790 50  0001 C CNN
 F 4 "CLOCK" H 2440 6790 50  0001 C CNN "Optional"
+F 5 "C" H 2440 6790 50  0001 C CNN "EMI_FILTER_TYPE"
 	1    2440 6790
 	1    0    0    -1
@@
 F 3 "~" H 2880 6800 50  0001 C CNN
 F 4 "CLOCK" H 2880 6800 50  0001 C CNN "Optional"
+F 5 "C" H 2880 6800 50  0001 C CNN "EMI_FILTER_TYPE"
 	1    2880 6800
 	1    0    0    -1
@@
 F 3 "http://www.murata.com/~/media/webrenewal/support/library/catalog/products/emc/emifil/c31e.ashx?la=en-gb" V 9690 2870 50  0001 C CNN
 F 4 "CLOCK" H 9690 2870 50  0001 C CNN "Optional"
+F 5 "W/FERRITE" H 9690 2870 50  0001 C CNN "EMI_FILTER_TYPE"
 	1    9690 2870
 	0    1    1    0
@@
 F 3 "http://www.murata.com/~/media/webrenewal/support/library/catalog/products/emc/emifil/c31e.ashx?la=en-gb" V 5390 4050 50  0001 C CNN
 F 4 "CLOCK" H 5390 4050 50  0001 C CNN "Optional"
+F 5 "R" H 5390 4050 50  0001 C CNN "EMI_FILTER_TYPE"
 	1    5390 4050
 	1    0    0    -1
@@
 F 3 "http://www.murata.com/~/media/webrenewal/support/library/catalog/products/emc/emifil/c31e.ashx?la=en-gb" V 5390 4450 50  0001 C CNN
 F 4 "CLOCK" H 5390 4450 50  0001 C CNN "Optional"
+F 5 "R" H 5390 4450 50  0001 C CNN "EMI_FILTER_TYPE"
 	1    5390 4450
 	1    0    0    -1

Commit message: Add part numbers for EMI filters Not the original filters, but what seem to be suitable replacements available today
Parts:
- E407: Cost (none) -> 0.234; MFG Name (none) -> MURATA; MFG Part Num (none) -> DSS1NB32A151Q91A
Changed lines of the file:
@@
 F 4 "CLOCK" H 9690 2870 50  0001 C CNN "Optional"
 F 5 "W/FERRITE" H 9690 2870 50  0001 C CNN "EMI_FILTER_TYPE"
+F 6 "0.234" H 9690 2870 50  0001 C CNN "Cost"
+F 7 "MURATA" H 9690 2870 50  0001 C CNN "MFG Name"
+F 8 "DSS1NB32A151Q91A" H 9690 2870 50  0001 C CNN "MFG Part Num"
 	1    9690 2870
 	0    1    1    0

Commit message: Add EMI filter 3D models, add logo, re-add Rock Lobster (closes #15) Thanks to Szabó Zoltán and Workshopshed!
Parts:
- E407: MFG Part Num DSS1NB32A151Q91A -> DSS1NB32A103Q91A
Changed lines of the file:
@@
 F 6 "0.234" H 9690 2870 50  0001 C CNN "Cost"
 F 7 "MURATA" H 9690 2870 50  0001 C CNN "MFG Name"
-F 8 "DSS1NB32A151Q91A" H 9690 2870 50  0001 C CNN "MFG Part Num"
+F 8 "DSS1NB32A103Q91A" H 9690 2870 50  0001 C CNN "MFG Part Num"
 	1    9690 2870
 	0    1    1    0

Commit message: (Try to) Identify the minimum set of required components
Parts:
- C33: Required (none) -> R
- E104, E105, E407, RP103, U33: Required (none) -> Y
Changed lines of the file:
@@
 F 4 "CLOCK" H 3640 2550 50  0001 C CNN "Optional"
 F 5 "N/A" H 3640 2550 50  0001 C CNN "MFG Name"
+F 6 "Y" H 3640 2550 50  0001 C CNN "Required"
 	1    3640 2550
 	1    0    0    -1
@@
 F 4 "CLOCK" H 3640 3950 50  0001 C CNN "Optional"
 F 5 "N/A" H 3640 3950 50  0001 C CNN "MFG Name"
+F 6 "Y" H 3640 3950 50  0001 C CNN "Required"
 	2    3640 3950
 	1    0    0    -1
@@
 F 4 "CLOCK" H 3640 3250 50  0001 C CNN "Optional"
 F 5 "N/A" H 3640 3250 50  0001 C CNN "MFG Name"
+F 6 "Y" H 3640 3250 50  0001 C CNN "Required"
 	3    3640 3250
 	1    0    0    -1
@@
 F 3 "~" H 5240 3250 50  0001 C CNN
 F 4 "CLOCK" H 5240 3250 50  0001 C CNN "Optional"
+F 5 "Y" H 5240 3250 50  0001 C CNN "Required"
 	1    5240 3250
 	0    1    1    0
@@
 F 4 "CLOCK" H 9790 3770 50  0001 C CNN "Optional"
 F 5 "N/A" H 9790 3770 50  0001 C CNN "MFG Name"
+F 6 "Y" H 9790 3770 50  0001 C CNN "Required"
 	5    9790 3770
 	1    0    0    -1
@@
 F 6 "0.071" H 10190 3870 50  0001 C CNN "Cost"
 F 7 "CLOCK" H 10190 3870 50  0001 C CNN "Optional"
+F 8 "R" H 10190 3870 50  0001 C CNN "Required"
 	1    10190 3870
 	1    0    0    -1
@@
 F 7 "MURATA" H 9690 2870 50  0001 C CNN "MFG Name"
 F 8 "DSS1NB32A103Q91A" H 9690 2870 50  0001 C CNN "MFG Part Num"
+F 9 "Y" H 9690 2870 50  0001 C CNN "Required"
 	1    9690 2870
 	0    1    1    0
@@
 F 4 "CLOCK" H 5390 4050 50  0001 C CNN "Optional"
 F 5 "R" H 5390 4050 50  0001 C CNN "EMI_FILTER_TYPE"
+F 6 "Y" H 5390 4050 50  0001 C CNN "Required"
 	1    5390 4050
 	1    0    0    -1
@@
 F 4 "CLOCK" H 5390 4450 50  0001 C CNN "Optional"
 F 5 "R" H 5390 4450 50  0001 C CNN "EMI_FILTER_TYPE"
+F 6 "Y" H 5390 4450 50  0001 C CNN "Required"
 	1    5390 4450
 	1    0    0    -1

Commit message: Rename "Optional" Field to "Section"
Parts:
- C33, E102, E103, E104, E105, E106, E107, E108, E109, E407, E791, E792, E793, E794, RP103, U33: Optional CLOCK -> (none); Section (none) -> CLOCK
Changed lines of the file:
@@
 F 2 "Package_DIP:DIP-16_W7.62mm_Socket_LongPads" H 3640 2550 50  0001 C CNN
 F 3 "http://www.ti.com/lit/gpn/sn74LS258" H 3640 2550 50  0001 C CNN
-F 4 "CLOCK" H 3640 2550 50  0001 C CNN "Optional"
+F 4 "CLOCK" H 3640 2550 50  0001 C CNN "Section"
 F 5 "N/A" H 3640 2550 50  0001 C CNN "MFG Name"
 F 6 "Y" H 3640 2550 50  0001 C CNN "Required"
@@
 F 2 "Package_DIP:DIP-16_W7.62mm_Socket_LongPads" H 6740 1650 50  0001 C CNN
 F 3 "http://www.ti.com/lit/gpn/sn74LS258" H 6740 1650 50  0001 C CNN
-F 4 "CLOCK" H 3640 3950 50  0001 C CNN "Optional"
+F 4 "CLOCK" H 3640 3950 50  0001 C CNN "Section"
 F 5 "N/A" H 3640 3950 50  0001 C CNN "MFG Name"
 F 6 "Y" H 3640 3950 50  0001 C CNN "Required"
@@
 F 2 "Package_DIP:DIP-16_W7.62mm_Socket_LongPads" H 6740 950 50  0001 C CNN
 F 3 "http://www.ti.com/lit/gpn/sn74LS258" H 6740 950 50  0001 C CNN
-F 4 "CLOCK" H 3640 3250 50  0001 C CNN "Optional"
+F 4 "CLOCK" H 3640 3250 50  0001 C CNN "Section"
 F 5 "N/A" H 3640 3250 50  0001 C CNN "MFG Name"
 F 6 "Y" H 3640 3250 50  0001 C CNN "Required"
@@
 F 2 "Resistor_THT:R_Array_SIP10" V 5615 3250 50  0001 C CNN
 F 3 "~" H 5240 3250 50  0001 C CNN
-F 4 "CLOCK" H 5240 3250 50  0001 C CNN "Optional"
+F 4 "CLOCK" H 5240 3250 50  0001 C CNN "Section"
 F 5 "Y" H 5240 3250 50  0001 C CNN "Required"
 	1    5240 3250
@@
 F 2 "Package_DIP:DIP-16_W7.62mm_Socket_LongPads" H 12890 1470 50  0001 C CNN
 F 3 "http://www.ti.com/lit/gpn/sn74LS258" H 12890 1470 50  0001 C CNN
-F 4 "CLOCK" H 9790 3770 50  0001 C CNN "Optional"
+F 4 "CLOCK" H 9790 3770 50  0001 C CNN "Section"
 F 5 "N/A" H 9790 3770 50  0001 C CNN "MFG Name"
 F 6 "Y" H 9790 3770 50  0001 C CNN "Required"
@@
 F 5 "C410C103K1H5TAAUTO" H 10190 3870 50  0001 C CNN "MFG Part Num"
 F 6 "0.071" H 10190 3870 50  0001 C CNN "Cost"
-F 7 "CLOCK" H 10190 3870 50  0001 C CNN "Optional"
+F 7 "CLOCK" H 10190 3870 50  0001 C CNN "Section"
 F 8 "R" H 10190 3870 50  0001 C CNN "Required"
 	1    10190 3870
@@
 F 2 "Raemixx500:C_Axial_L6.3mm_D2.5mm_P10.16mm" H 6148 4620 50  0001 C CNN
 F 3 "~" H 6110 4770 50  0001 C CNN
-F 4 "CLOCK" H 6110 4770 50  0001 C CNN "Optional"
+F 4 "CLOCK" H 6110 4770 50  0001 C CNN "Section"
 F 5 "C" H 6110 4770 50  0001 C CNN "EMI_FILTER_TYPE"
 	1    6110 4770
@@
 F 2 "Raemixx500:C_Axial_L6.3mm_D2.5mm_P10.16mm" H 6588 4630 50  0001 C CNN
 F 3 "~" H 6550 4780 50  0001 C CNN
-F 4 "CLOCK" H 6550 4780 50  0001 C CNN "Optional"
+F 4 "CLOCK" H 6550 4780 50  0001 C CNN "Section"
 F 5 "C" H 6550 4780 50  0001 C CNN "EMI_FILTER_TYPE"
 	1    6550 4780
@@
 F 2 "Raemixx500:C_Axial_L6.3mm_D2.5mm_P10.16mm" H 7028 4630 50  0001 C CNN
 F 3 "~" H 6990 4780 50  0001 C CNN
-F 4 "CLOCK" H 6990 4780 50  0001 C CNN "Optional"
+F 4 "CLOCK" H 6990 4780 50  0001 C CNN "Section"
 F 5 "C" H 6990 4780 50  0001 C CNN "EMI_FILTER_TYPE"
 	1    6990 4780
@@
 F 2 "Raemixx500:C_Axial_L6.3mm_D2.5mm_P10.16mm" H 7468 4640 50  0001 C CNN
 F 3 "~" H 7430 4790 50  0001 C CNN
-F 4 "CLOCK" H 7430 4790 50  0001 C CNN "Optional"
+F 4 "CLOCK" H 7430 4790 50  0001 C CNN "Section"
 F 5 "C" H 7430 4790 50  0001 C CNN "EMI_FILTER_TYPE"
 	1    7430 4790
@@
 F 2 "Raemixx500:C_Axial_L9.0mm_D3.2mm_P12.70mm" H 7908 4640 50  0001 C CNN
 F 3 "~" H 7870 4790 50  0001 C CNN
-F 4 "CLOCK" H 7870 4790 50  0001 C CNN "Optional"
+F 4 "CLOCK" H 7870 4790 50  0001 C CNN "Section"
 F 5 "C" H 7870 4790 50  0001 C CNN "EMI_FILTER_TYPE"
 	1    7870 4790
@@
 F 2 "Raemixx500:C_Axial_L9.0mm_D3.2mm_P12.70mm" H 2038 4610 50  0001 C CNN
 F 3 "~" H 2000 4760 50  0001 C CNN
-F 4 "CLOCK" H 2000 4760 50  0001 C CNN "Optional"
+F 4 "CLOCK" H 2000 4760 50  0001 C CNN "Section"
 F 5 "C" H 2000 4760 50  0001 C CNN "EMI_FILTER_TYPE"
 	1    2000 4760
@@
 F 2 "Raemixx500:C_Axial_L9.0mm_D3.2mm_P12.70mm" H 2478 4620 50  0001 C CNN
 F 3 "~" H 2440 4770 50  0001 C CNN
-F 4 "CLOCK" H 2440 4770 50  0001 C CNN "Optional"
+F 4 "CLOCK" H 2440 4770 50  0001 C CNN "Section"
 F 5 "C" H 2440 4770 50  0001 C CNN "EMI_FILTER_TYPE"
 	1    2440 4770
@@
 F 2 "Raemixx500:C_Axial_L9.0mm_D3.2mm_P12.70mm" H 2918 4620 50  0001 C CNN
 F 3 "~" H 2880 4770 50  0001 C CNN
-F 4 "CLOCK" H 2880 4770 50  0001 C CNN "Optional"
+F 4 "CLOCK" H 2880 4770 50  0001 C CNN "Section"
 F 5 "C" H 2880 4770 50  0001 C CNN "EMI_FILTER_TYPE"
 	1    2880 4770
@@
 F 2 "Raemixx500:C_Axial_L6.3mm_D2.5mm_P10.16mm" H 2478 6640 50  0001 C CNN
 F 3 "~" H 2440 6790 50  0001 C CNN
-F 4 "CLOCK" H 2440 6790 50  0001 C CNN "Optional"
+F 4 "CLOCK" H 2440 6790 50  0001 C CNN "Section"
 F 5 "C" H 2440 6790 50  0001 C CNN "EMI_FILTER_TYPE"
 	1    2440 6790
@@
 F 2 "Raemixx500:C_Axial_L9.0mm_D3.2mm_P12.70mm" H 2918 6650 50  0001 C CNN
 F 3 "~" H 2880 6800 50  0001 C CNN
-F 4 "CLOCK" H 2880 6800 50  0001 C CNN "Optional"
+F 4 "CLOCK" H 2880 6800 50  0001 C CNN "Section"
 F 5 "C" H 2880 6800 50  0001 C CNN "EMI_FILTER_TYPE"
 	1    2880 6800
@@
 F 2 "Raemixx500:EMI_Filter_Short" V 9690 2870 50  0001 C CNN
 F 3 "http://www.murata.com/~/media/webrenewal/support/library/catalog/products/emc/emifil/c31e.ashx?la=en-gb" V 9690 2870 50  0001 C CNN
-F 4 "CLOCK" H 9690 2870 50  0001 C CNN "Optional"
+F 4 "CLOCK" H 9690 2870 50  0001 C CNN "Section"
 F 5 "W/FERRITE" H 9690 2870 50  0001 C CNN "EMI_FILTER_TYPE"
 F 6 "0.234" H 9690 2870 50  0001 C CNN "Cost"
@@
 F 2 "Raemixx500:EMI_Filter_Long" V 5390 4050 50  0001 C CNN
 F 3 "http://www.murata.com/~/media/webrenewal/support/library/catalog/products/emc/emifil/c31e.ashx?la=en-gb" V 5390 4050 50  0001 C CNN
-F 4 "CLOCK" H 5390 4050 50  0001 C CNN "Optional"
+F 4 "CLOCK" H 5390 4050 50  0001 C CNN "Section"
 F 5 "R" H 5390 4050 50  0001 C CNN "EMI_FILTER_TYPE"
 F 6 "Y" H 5390 4050 50  0001 C CNN "Required"
@@
 F 2 "Raemixx500:EMI_Filter_Long" V 5390 4450 50  0001 C CNN
 F 3 "http://www.murata.com/~/media/webrenewal/support/library/catalog/products/emc/emifil/c31e.ashx?la=en-gb" V 5390 4450 50  0001 C CNN
-F 4 "CLOCK" H 5390 4450 50  0001 C CNN "Optional"
+F 4 "CLOCK" H 5390 4450 50  0001 C CNN "Section"
 F 5 "R" H 5390 4450 50  0001 C CNN "EMI_FILTER_TYPE"
 F 6 "Y" H 5390 4450 50  0001 C CNN "Required"
