File: ram.sch (KiCad schematic (older format))
At the start: 25 parts, among them U16 XX4256, U17 XX4256, U18 XX4256, U19 XX4256, U20 XX4256, U21 XX4256, U22 XX4256, U23 XX4256, U32 74LS139, U34 74LS373, U35 74LS244

Commit message: Rename "Optional" Field to "Section"
Parts:
- C16, C17, C18, C19, C20, R201, R202, RP201, RP202, RP203, U16, U17, U18, U19, U20, U21, U22, U23, U32, U34, U35: Optional MEMORY -> (none); Section (none) -> MEMORY
- JP3A1, JP3B1, JP4A1, JP4B1: Optional JMP -> (none); Section (none) -> JMP
Changed lines of the file:
@@
 F 2 "Package_DIP:DIP-20_W7.62mm_Socket_LongPads" H 3100 2095 50  0001 C CNN
 F 3 "http://www.ti.com/lit/gpn/sn74LS373" H 3100 2095 50  0001 C CNN
-F 4 "MEMORY" H 3100 2095 50  0001 C CNN "Optional"
+F 4 "MEMORY" H 3100 2095 50  0001 C CNN "Section"
 F 5 "0.68" H 3100 2095 50  0001 C CNN "Cost"
 F 6 "TI" H 3100 2095 50  0001 C CNN "MFG Name"
@@
 F 2 "Package_DIP:DIP-20_W7.62mm_Socket_LongPads" H 3100 3625 50  0001 C CNN
 F 3 "http://www.ti.com/lit/gpn/sn74LS244" H 3100 3625 50  0001 C CNN
-F 4 "MEMORY" H 3100 3625 50  0001 C CNN "Optional"
+F 4 "MEMORY" H 3100 3625 50  0001 C CNN "Section"
 F 5 "0.62" H 3100 3625 50  0001 C CNN "Cost"
 F 6 "TI" H 3100 3625 50  0001 C CNN "MFG Name"
@@
 F 2 "Resistor_THT:R_Array_SIP10" V 6265 2280 50  0001 C CNN
 F 3 "http://www.vishay.com/docs/31509/csc.pdf" H 5390 2280 50  0001 C CNN
-F 4 "MEMORY" H 5390 2280 50  0001 C CNN "Optional"
+F 4 "MEMORY" H 5390 2280 50  0001 C CNN "Section"
 F 5 "Y" H 5390 2280 50  0001 C CNN "Required"
 	1    5390 2280
@@
 F 2 "Resistor_THT:R_Array_SIP10" V 6265 3830 50  0001 C CNN
 F 3 "http://www.vishay.com/docs/31509/csc.pdf" H 5390 3830 50  0001 C CNN
-F 4 "MEMORY" H 5390 3830 50  0001 C CNN "Optional"
+F 4 "MEMORY" H 5390 3830 50  0001 C CNN "Section"
 F 5 "Y" H 5390 3830 50  0001 C CNN "Required"
 	1    5390 3830
@@
 F 2 "Resistor_THT:R_Array_SIP10" V 6265 5940 50  0001 C CNN
 F 3 "http://www.vishay.com/docs/31509/csc.pdf" H 5390 5940 50  0001 C CNN
-F 4 "MEMORY" H 5390 5940 50  0001 C CNN "Optional"
+F 4 "MEMORY" H 5390 5940 50  0001 C CNN "Section"
 F 5 "Y" H 5390 5940 50  0001 C CNN "Required"
 	1    5390 5940
@@
 F 2 "Package_DIP:DIP-16_W7.62mm_Socket_LongPads" H 5165 7570 50  0001 C CNN
 F 3 "http://www.ti.com/lit/gpn/sn74LS139" H 5165 7570 50  0001 C CNN
-F 4 "MEMORY" H 5165 7570 50  0001 C CNN "Optional"
+F 4 "MEMORY" H 5165 7570 50  0001 C CNN "Section"
 F 5 "0.615" H 5165 7570 50  0001 C CNN "Cost"
 F 6 "TI" H 5165 7570 50  0001 C CNN "MFG Name"
@@
 F 2 "Package_DIP:DIP-16_W7.62mm_Socket_LongPads" H 5165 8360 50  0001 C CNN
 F 3 "http://www.ti.com/lit/gpn/sn74LS139" H 5165 8360 50  0001 C CNN
-F 4 "MEMORY" H 5165 8360 50  0001 C CNN "Optional"
+F 4 "MEMORY" H 5165 8360 50  0001 C CNN "Section"
 F 5 "0.615" H 5165 8360 50  0001 C CNN "Cost"
 F 6 "TI" H 5165 8360 50  0001 C CNN "MFG Name"
@@
 F 4 "SKIP" H 4850 4980 50  0001 C CNN "MFG Name"
 F 5 "SKIP" H 4850 4980 50  0001 C CNN "MFG Part Num"
-F 6 "JMP" H 4850 4980 50  0001 C CNN "Optional"
+F 6 "JMP" H 4850 4980 50  0001 C CNN "Section"
 	1    4850 4980
 	1    0    0    -1
@@
 F 4 "SKIP" H 4850 5190 50  0001 C CNN "MFG Name"
 F 5 "SKIP" H 4850 5190 50  0001 C CNN "MFG Part Num"
-F 6 "JMP" H 4850 5190 50  0001 C CNN "Optional"
+F 6 "JMP" H 4850 5190 50  0001 C CNN "Section"
 	1    4850 5190
 	1    0    0    -1
@@
 F 2 "Raemixx500:R_Axial_DIN0309_L9.0mm_D3.2mm_P12.70mm_Horizontal" V 7740 1665 50  0001 C CNN
 F 3 "~" H 7810 1665 50  0001 C CNN
-F 4 "MEMORY" H 7810 1665 50  0001 C CNN "Optional"
+F 4 "MEMORY" H 7810 1665 50  0001 C CNN "Section"
 F 5 "Y" H 7810 1665 50  0001 C CNN "Required"
 	1    7810 1665
@@
 F 2 "Raemixx500:R_Axial_DIN0309_L9.0mm_D3.2mm_P12.70mm_Horizontal" V 8090 3785 50  0001 C CNN
 F 3 "~" H 8160 3785 50  0001 C CNN
-F 4 "MEMORY" H 8160 3785 50  0001 C CNN "Optional"
+F 4 "MEMORY" H 8160 3785 50  0001 C CNN "Section"
 F 5 "Y" H 8160 3785 50  0001 C CNN "Required"
 	1    8160 3785
@@
 F 2 "Package_DIP:DIP-20_W7.62mm_Socket_LongPads" H 9300 1700 50  0001 C CNN
 F 3 "DOCUMENTATION" H 9300 1700 50  0001 C CNN
-F 4 "MEMORY" H 9300 1700 50  0001 C CNN "Optional"
+F 4 "MEMORY" H 9300 1700 50  0001 C CNN "Section"
 F 5 "Y" H 9300 1700 50  0001 C CNN "Required"
 	1    9300 1700
@@
 F 2 "Package_DIP:DIP-20_W7.62mm_Socket_LongPads" H 10975 1700 50  0001 C CNN
 F 3 "DOCUMENTATION" H 10975 1700 50  0001 C CNN
-F 4 "MEMORY" H 10975 1700 50  0001 C CNN "Optional"
+F 4 "MEMORY" H 10975 1700 50  0001 C CNN "Section"
 F 5 "Y" H 10975 1700 50  0001 C CNN "Required"
 	1    10975 1700
@@
 F 2 "Package_DIP:DIP-20_W7.62mm_Socket_LongPads" H 12650 1700 50  0001 C CNN
 F 3 "DOCUMENTATION" H 12650 1700 50  0001 C CNN
-F 4 "MEMORY" H 12650 1700 50  0001 C CNN "Optional"
+F 4 "MEMORY" H 12650 1700 50  0001 C CNN "Section"
 F 5 "Y" H 12650 1700 50  0001 C CNN "Required"
 	1    12650 1700
@@
 F 2 "Package_DIP:DIP-20_W7.62mm_Socket_LongPads" H 14325 1700 50  0001 C CNN
 F 3 "DOCUMENTATION" H 14325 1700 50  0001 C CNN
-F 4 "MEMORY" H 14325 1700 50  0001 C CNN "Optional"
+F 4 "MEMORY" H 14325 1700 50  0001 C CNN "Section"
 F 5 "Y" H 14325 1700 50  0001 C CNN "Required"
 	1    14325 1700
@@
 F 2 "Package_DIP:DIP-20_W7.62mm_Socket_LongPads" H 9300 3980 50  0001 C CNN
 F 3 "DOCUMENTATION" H 9300 3980 50  0001 C CNN
-F 4 "MEMORY" H 9300 3980 50  0001 C CNN "Optional"
+F 4 "MEMORY" H 9300 3980 50  0001 C CNN "Section"
 	1    9300 3980
 	1    0    0    -1
@@
 F 2 "Package_DIP:DIP-20_W7.62mm_Socket_LongPads" H 10975 3980 50  0001 C CNN
 F 3 "DOCUMENTATION" H 10975 3980 50  0001 C CNN
-F 4 "MEMORY" H 10975 3980 50  0001 C CNN "Optional"
+F 4 "MEMORY" H 10975 3980 50  0001 C CNN "Section"
 	1    10975 3980
 	1    0    0    -1
@@
 F 2 "Package_DIP:DIP-20_W7.62mm_Socket_LongPads" H 12650 3980 50  0001 C CNN
 F 3 "DOCUMENTATION" H 12650 3980 50  0001 C CNN
-F 4 "MEMORY" H 12650 3980 50  0001 C CNN "Optional"
+F 4 "MEMORY" H 12650 3980 50  0001 C CNN "Section"
 	1    12650 3980
 	1    0    0    -1
@@
 F 2 "Package_DIP:DIP-20_W7.62mm_Socket_LongPads" H 14325 3980 50  0001 C CNN
 F 3 "DOCUMENTATION" H 14325 3980 50  0001 C CNN
-F 4 "MEMORY" H 14325 3980 50  0001 C CNN "Optional"
+F 4 "MEMORY" H 14325 3980 50  0001 C CNN "Section"
 	1    14325 3980
 	1    0    0    -1
@@
 F 4 "SKIP" H 7185 7470 50  0001 C CNN "MFG Name"
 F 5 "SKIP" H 7185 7470 50  0001 C CNN "MFG Part Num"
-F 6 "JMP" H 7185 7470 50  0001 C CNN "Optional"
+F 6 "JMP" H 7185 7470 50  0001 C CNN "Section"
 F 7 "Y" H 7185 7470 50  0001 C CNN "Required"
 	1    7185 7470
@@
 F 4 "SKIP" H 7185 8260 50  0001 C CNN "MFG Name"
 F 5 "SKIP" H 7185 8260 50  0001 C CNN "MFG Part Num"
-F 6 "JMP" H 7185 8260 50  0001 C CNN "Optional"
+F 6 "JMP" H 7185 8260 50  0001 C CNN "Section"
 F 7 "Y" H 7185 8260 50  0001 C CNN "Required"
 	1    7185 8260
@@
 F 2 "Package_DIP:DIP-20_W7.62mm_Socket_LongPads" H 12095 7125 50  0001 C CNN
 F 3 "DOCUMENTATION" H 12095 7125 50  0001 C CNN
-F 4 "MEMORY" H 12095 7125 50  0001 C CNN "Optional"
+F 4 "MEMORY" H 12095 7125 50  0001 C CNN "Section"
 F 5 "Y" H 12095 7125 50  0001 C CNN "Required"
 	2    12095 7125
@@
 F 2 "Package_DIP:DIP-20_W7.62mm_Socket_LongPads" H 12980 7125 50  0001 C CNN
 F 3 "DOCUMENTATION" H 12980 7125 50  0001 C CNN
-F 4 "MEMORY" H 12980 7125 50  0001 C CNN "Optional"
+F 4 "MEMORY" H 12980 7125 50  0001 C CNN "Section"
 	2    12980 7125
 	1    0    0    -1
@@
 F 5 "C412C334M5U5TA" H 11465 7130 50  0001 C CNN "MFG Part Num"
 F 6 "0.078" H 11465 7130 50  0001 C CNN "Cost"
-F 7 "MEMORY" H 11465 7130 50  0001 C CNN "Optional"
+F 7 "MEMORY" H 11465 7130 50  0001 C CNN "Section"
 F 8 "R" H 11465 7130 50  0001 C CNN "Required"
 	1    11465 7130
@@
 F 2 "Package_DIP:DIP-20_W7.62mm_Socket_LongPads" H 14510 7125 50  0001 C CNN
 F 3 "DOCUMENTATION" H 14510 7125 50  0001 C CNN
-F 4 "MEMORY" H 14510 7125 50  0001 C CNN "Optional"
+F 4 "MEMORY" H 14510 7125 50  0001 C CNN "Section"
 F 5 "Y" H 14510 7125 50  0001 C CNN "Required"
 	2    14510 7125
@@
 F 2 "Package_DIP:DIP-20_W7.62mm_Socket_LongPads" H 15395 7125 50  0001 C CNN
 F 3 "DOCUMENTATION" H 15395 7125 50  0001 C CNN
-F 4 "MEMORY" H 15395 7125 50  0001 C CNN "Optional"
+F 4 "MEMORY" H 15395 7125 50  0001 C CNN "Section"
 	2    15395 7125
 	1    0    0    -1
@@
 F 5 "C412C334M5U5TA" H 13880 7130 50  0001 C CNN "MFG Part Num"
 F 6 "0.078" H 13880 7130 50  0001 C CNN "Cost"
-F 7 "MEMORY" H 13880 7130 50  0001 C CNN "Optional"
+F 7 "MEMORY" H 13880 7130 50  0001 C CNN "Section"
 F 8 "R" H 13880 7130 50  0001 C CNN "Required"
 	1    13880 7130
@@
 F 5 "C412C334M5U5TA" H 15425 8910 50  0001 C CNN "MFG Part Num"
 F 6 "0.078" H 15425 8910 50  0001 C CNN "Cost"
-F 7 "MEMORY" H 15425 8910 50  0001 C CNN "Optional"
+F 7 "MEMORY" H 15425 8910 50  0001 C CNN "Section"
 F 8 "R" H 15425 8910 50  0001 C CNN "Required"
 	1    15425 8910
@@
 F 2 "Package_DIP:DIP-20_W7.62mm_Socket_LongPads" H 11210 8905 50  0001 C CNN
 F 3 "DOCUMENTATION" H 11210 8905 50  0001 C CNN
-F 4 "MEMORY" H 11210 8905 50  0001 C CNN "Optional"
+F 4 "MEMORY" H 11210 8905 50  0001 C CNN "Section"
 F 5 "Y" H 11210 8905 50  0001 C CNN "Required"
 	2    11210 8905
@@
 F 2 "Package_DIP:DIP-20_W7.62mm_Socket_LongPads" H 12095 8905 50  0001 C CNN
 F 3 "DOCUMENTATION" H 12095 8905 50  0001 C CNN
-F 4 "MEMORY" H 12095 8905 50  0001 C CNN "Optional"
+F 4 "MEMORY" H 12095 8905 50  0001 C CNN "Section"
 	2    12095 8905
 	1    0    0    -1
@@
 F 5 "C412C334M5U5TA" H 10580 8910 50  0001 C CNN "MFG Part Num"
 F 6 "0.078" H 10580 8910 50  0001 C CNN "Cost"
-F 7 "MEMORY" H 10580 8910 50  0001 C CNN "Optional"
+F 7 "MEMORY" H 10580 8910 50  0001 C CNN "Section"
 F 8 "R" H 10580 8910 50  0001 C CNN "Required"
 	1    10580 8910
@@
 F 2 "Package_DIP:DIP-20_W7.62mm_Socket_LongPads" H 13625 8905 50  0001 C CNN
 F 3 "DOCUMENTATION" H 13625 8905 50  0001 C CNN
-F 4 "MEMORY" H 13625 8905 50  0001 C CNN "Optional"
+F 4 "MEMORY" H 13625 8905 50  0001 C CNN "Section"
 F 5 "Y" H 13625 8905 50  0001 C CNN "Required"
 	2    13625 8905
@@
 F 2 "Package_DIP:DIP-20_W7.62mm_Socket_LongPads" H 14510 8905 50  0001 C CNN
 F 3 "DOCUMENTATION" H 14510 8905 50  0001 C CNN
-F 4 "MEMORY" H 14510 8905 50  0001 C CNN "Optional"
+F 4 "MEMORY" H 14510 8905 50  0001 C CNN "Section"
 	2    14510 8905
 	1    0    0    -1
@@
 F 5 "C412C334M5U5TA" H 12995 8910 50  0001 C CNN "MFG Part Num"
 F 6 "0.078" H 12995 8910 50  0001 C CNN "Cost"
-F 7 "MEMORY" H 12995 8910 50  0001 C CNN "Optional"
+F 7 "MEMORY" H 12995 8910 50  0001 C CNN "Section"
 F 8 "R" H 12995 8910 50  0001 C CNN "Required"
 	1    12995 8910
