File: rtc.sch (KiCad schematic (older format))
At the start: 16 parts, among them U36 74LS05, U9 MSM6242B, Y9 32768 Hz

Commit message: Begin adding part numbers
Parts:
- BT9, C913, D911, D912, D913, TC9, U9, Y9: Optional (none) -> RTC
- C9: Cost (none) -> 0.078; MFG Name (none) -> KEMET; MFG Part Num (none) -> C412C334M5U5TA; Optional (none) -> RTC
- C911: Cost (none) -> 0.141; MFG Name (none) -> AVX; MFG Part Num (none) -> SA102A220JARC
- JP9: MFG Name (none) -> SKIP; MFG Part Num (none) -> SKIP; Optional (none) -> JMP
- U36: Optional (none) -> FLOPPY/RTC
Changed lines of the file:
@@
 F 2 "Package_DIP:DIP-18_W7.62mm_Socket_LongPads" H 7995 2125 50  0001 C CNN
 F 3 "DOCUMENTATION" H 7995 2125 50  0001 C CNN
+F 4 "RTC" H 7995 2125 50  0001 C CNN "Optional"
 	1    7995 2125
 	1    0    0    -1
@@
 F 2 "Package_DIP:DIP-14_W7.62mm_Socket_LongPads" H 4680 2525 50  0001 C CNN
 F 3 "http://www.ti.com/lit/gpn/sn74LS05" H 4680 2525 50  0001 C CNN
+F 4 "FLOPPY/RTC" H 4680 2525 50  0001 C CNN "Optional"
 	5    4680 2525
 	1    0    0    -1
@@
 F 2 "Raemixx500:Jumper2-Open" H 4015 3025 50  0001 C CNN
 F 3 "~" H 4015 3025 50  0001 C CNN
+F 4 "SKIP" H 4015 3025 50  0001 C CNN "MFG Name"
+F 5 "SKIP" H 4015 3025 50  0001 C CNN "MFG Part Num"
+F 6 "JMP" H 4015 3025 50  0001 C CNN "Optional"
 	1    4015 3025
 	0    -1   -1   0
@@
 F 2 "Raemixx500:VariCap" H 9640 2325 50  0001 C CNN
 F 3 "~" H 9640 2325 50  0001 C CNN
+F 4 "RTC" H 9640 2325 50  0001 C CNN "Optional"
 	1    9640 2325
 	0    -1   -1   0
@@
 F 2 "Raemixx500:C_Axial_L6.3mm_D2.5mm_P10.16mm" H 9678 2575 50  0001 C CNN
 F 3 "~" H 9640 2725 50  0001 C CNN
+F 4 "0.141" H 9640 2725 50  0001 C CNN "Cost"
+F 5 "AVX" H 9640 2725 50  0001 C CNN "MFG Name"
+F 6 "SA102A220JARC" H 9640 2725 50  0001 C CNN "MFG Part Num"
 	1    9640 2725
 	0    1    1    0
@@
 F 2 "Package_DIP:DIP-14_W7.62mm_Socket_LongPads" H 3170 2525 50  0001 C CNN
 F 3 "http://www.ti.com/lit/gpn/sn74LS05" H 3170 2525 50  0001 C CNN
+F 4 "FLOPPY/RTC" H 3170 2525 50  0001 C CNN "Optional"
 	6    3170 2525
 	1    0    0    -1
@@
 F 2 "Raemixx500:Crystal_RTC" H 9175 2525 50  0001 C CNN
 F 3 "~" H 9175 2525 50  0001 C CNN
+F 4 "RTC" H 9175 2525 50  0001 C CNN "Optional"
 	1    9175 2525
 	0    1    1    0
@@
 F 2 "Raemixx500:Battery_Holder_Coin_2032_BS-7" V 2950 5930 50  0001 C CNN
 F 3 "~" V 2950 5930 50  0001 C CNN
+F 4 "RTC" H 2950 5870 50  0001 C CNN "Optional"
 	1    2950 5870
 	1    0    0    -1
@@
 F 2 "Capacitor_THT:CP_Radial_D8.0mm_P5.00mm" H 3805 5820 50  0001 C CNN
 F 3 "~" H 3805 5820 50  0001 C CNN
+F 4 "RTC" H 3805 5820 50  0001 C CNN "Optional"
 	1    3805 5820
 	1    0    0    -1
@@
 F 2 "Package_DIP:DIP-18_W7.62mm_Socket_LongPads" H 4555 6225 50  0001 C CNN
 F 3 "DOCUMENTATION" H 4555 6225 50  0001 C CNN
+F 4 "RTC" H 4555 5825 50  0001 C CNN "Optional"
 	2    4555 5825
 	1    0    0    -1
@@
 F 2 "Raemixx500:C_Axial_L6.3mm_D2.5mm_P10.16mm" H 5528 5670 50  0001 C CNN
 F 3 "~" H 5490 5820 50  0001 C CNN
+F 4 "KEMET" H 5490 5820 50  0001 C CNN "MFG Name"
+F 5 "C412C334M5U5TA" H 5490 5820 50  0001 C CNN "MFG Part Num"
+F 6 "0.078" H 5490 5820 50  0001 C CNN "Cost"
+F 7 "RTC" H 5490 5820 50  0001 C CNN "Optional"
 	1    5490 5820
 	1    0    0    -1
@@
 F 2 "Diode_THT:D_DO-35_SOD27_P12.70mm_Horizontal" H 3805 4720 50  0001 C CNN
 F 3 "~" H 3805 4720 50  0001 C CNN
+F 4 "RTC" H 3805 4720 50  0001 C CNN "Optional"
 	1    3805 4720
 	0    -1   -1   0
@@
 F 2 "Diode_THT:D_DO-35_SOD27_P12.70mm_Horizontal" H 4095 4430 50  0001 C CNN
 F 3 "~" H 4095 4430 50  0001 C CNN
+F 4 "RTC" H 4095 4430 50  0001 C CNN "Optional"
 	1    4095 4430
 	-1   0    0    1
@@
 F 2 "Diode_THT:D_DO-35_SOD27_P12.70mm_Horizontal" H 3365 5100 50  0001 C CNN
 F 3 "~" H 3365 5100 50  0001 C CNN
+F 4 "RTC" H 3365 5100 50  0001 C CNN "Optional"
 	1    3365 5100
 	-1   0    0    1

Commit message: More part numbers
Parts:
- C913: Cost (none) -> 0.41; MFG Name (none) -> RS PRO; MFG Part Num (none) -> 181-4685
- U36: Cost (none) -> 0.668; MFG Name (none) -> TI; MFG Part Num (none) -> SN74LS05N
Changed lines of the file:
@@
 F 3 "http://www.ti.com/lit/gpn/sn74LS05" H 4680 2525 50  0001 C CNN
 F 4 "FLOPPY/RTC" H 4680 2525 50  0001 C CNN "Optional"
+F 5 "0.668" H 4680 2525 50  0001 C CNN "Cost"
+F 6 "TI" H 4680 2525 50  0001 C CNN "MFG Name"
+F 7 "SN74LS05N" H 4680 2525 50  0001 C CNN "MFG Part Num"
 	5    4680 2525
 	1    0    0    -1
@@
 F 3 "http://www.ti.com/lit/gpn/sn74LS05" H 3170 2525 50  0001 C CNN
 F 4 "FLOPPY/RTC" H 3170 2525 50  0001 C CNN "Optional"
+F 5 "0.668" H 3170 2525 50  0001 C CNN "Cost"
+F 6 "TI" H 3170 2525 50  0001 C CNN "MFG Name"
+F 7 "SN74LS05N" H 3170 2525 50  0001 C CNN "MFG Part Num"
 	6    3170 2525
 	1    0    0    -1
@@
 F 3 "~" H 3805 5820 50  0001 C CNN
 F 4 "RTC" H 3805 5820 50  0001 C CNN "Optional"
+F 5 "0.41" H 3805 5820 50  0001 C CNN "Cost"
+F 6 "RS PRO" H 3805 5820 50  0001 C CNN "MFG Name"
+F 7 "181-4685" H 3805 5820 50  0001 C CNN "MFG Part Num"
 	1    3805 5820
 	1    0    0    -1

Commit message: Rename "Optional" Field to "Section"
Parts:
- BT9, C9, C913, D911, D912, D913, TC9, U9, Y9: Optional RTC -> (none); Section (none) -> RTC
- JP9: Optional JMP -> (none); Section (none) -> JMP
- U36: Optional FLOPPY/RTC -> (none); Section (none) -> FLOPPY/RTC
Changed lines of the file:
@@
 F 2 "Package_DIP:DIP-18_W7.62mm_Socket_LongPads" H 7995 2125 50  0001 C CNN
 F 3 "DOCUMENTATION" H 7995 2125 50  0001 C CNN
-F 4 "RTC" H 7995 2125 50  0001 C CNN "Optional"
+F 4 "RTC" H 7995 2125 50  0001 C CNN "Section"
 	1    7995 2125
 	1    0    0    -1
@@
 F 2 "Package_DIP:DIP-14_W7.62mm_Socket_LongPads" H 4680 2525 50  0001 C CNN
 F 3 "http://www.ti.com/lit/gpn/sn74LS05" H 4680 2525 50  0001 C CNN
-F 4 "FLOPPY/RTC" H 4680 2525 50  0001 C CNN "Optional"
+F 4 "FLOPPY/RTC" H 4680 2525 50  0001 C CNN "Section"
 F 5 "0.668" H 4680 2525 50  0001 C CNN "Cost"
 F 6 "TI" H 4680 2525 50  0001 C CNN "MFG Name"
@@
 F 4 "SKIP" H 4015 3025 50  0001 C CNN "MFG Name"
 F 5 "SKIP" H 4015 3025 50  0001 C CNN "MFG Part Num"
-F 6 "JMP" H 4015 3025 50  0001 C CNN "Optional"
+F 6 "JMP" H 4015 3025 50  0001 C CNN "Section"
 	1    4015 3025
 	0    -1   -1   0
@@
 F 2 "Raemixx500:VariCap" H 9640 2325 50  0001 C CNN
 F 3 "~" H 9640 2325 50  0001 C CNN
-F 4 "RTC" H 9640 2325 50  0001 C CNN "Optional"
+F 4 "RTC" H 9640 2325 50  0001 C CNN "Section"
 	1    9640 2325
 	0    -1   -1   0
@@
 F 2 "Package_DIP:DIP-14_W7.62mm_Socket_LongPads" H 3170 2525 50  0001 C CNN
 F 3 "http://www.ti.com/lit/gpn/sn74LS05" H 3170 2525 50  0001 C CNN
-F 4 "FLOPPY/RTC" H 3170 2525 50  0001 C CNN "Optional"
+F 4 "FLOPPY/RTC" H 3170 2525 50  0001 C CNN "Section"
 F 5 "0.668" H 3170 2525 50  0001 C CNN "Cost"
 F 6 "TI" H 3170 2525 50  0001 C CNN "MFG Name"
@@
 F 2 "Raemixx500:Crystal_RTC" H 9175 2525 50  0001 C CNN
 F 3 "~" H 9175 2525 50  0001 C CNN
-F 4 "RTC" H 9175 2525 50  0001 C CNN "Optional"
+F 4 "RTC" H 9175 2525 50  0001 C CNN "Section"
 	1    9175 2525
 	0    1    1    0
@@
 F 2 "Raemixx500:Battery_Holder_Coin_2032_BS-7" V 2950 5930 50  0001 C CNN
 F 3 "~" V 2950 5930 50  0001 C CNN
-F 4 "RTC" H 2950 5870 50  0001 C CNN "Optional"
+F 4 "RTC" H 2950 5870 50  0001 C CNN "Section"
 	1    2950 5870
 	1    0    0    -1
@@
 F 2 "Capacitor_THT:CP_Radial_D8.0mm_P5.00mm" H 3805 5820 50  0001 C CNN
 F 3 "~" H 3805 5820 50  0001 C CNN
-F 4 "RTC" H 3805 5820 50  0001 C CNN "Optional"
+F 4 "RTC" H 3805 5820 50  0001 C CNN "Section"
 F 5 "0.41" H 3805 5820 50  0001 C CNN "Cost"
 F 6 "RS PRO" H 3805 5820 50  0001 C CNN "MFG Name"
@@
 F 2 "Package_DIP:DIP-18_W7.62mm_Socket_LongPads" H 4555 6225 50  0001 C CNN
 F 3 "DOCUMENTATION" H 4555 6225 50  0001 C CNN
-F 4 "RTC" H 4555 5825 50  0001 C CNN "Optional"
+F 4 "RTC" H 4555 5825 50  0001 C CNN "Section"
 	2    4555 5825
 	1    0    0    -1
@@
 F 5 "C412C334M5U5TA" H 5490 5820 50  0001 C CNN "MFG Part Num"
 F 6 "0.078" H 5490 5820 50  0001 C CNN "Cost"
-F 7 "RTC" H 5490 5820 50  0001 C CNN "Optional"
+F 7 "RTC" H 5490 5820 50  0001 C CNN "Section"
 	1    5490 5820
 	1    0    0    -1
@@
 F 2 "Diode_THT:D_DO-35_SOD27_P12.70mm_Horizontal" H 3805 4720 50  0001 C CNN
 F 3 "~" H 3805 4720 50  0001 C CNN
-F 4 "RTC" H 3805 4720 50  0001 C CNN "Optional"
+F 4 "RTC" H 3805 4720 50  0001 C CNN "Section"
 	1    3805 4720
 	0    -1   -1   0
@@
 F 2 "Diode_THT:D_DO-35_SOD27_P12.70mm_Horizontal" H 4095 4430 50  0001 C CNN
 F 3 "~" H 4095 4430 50  0001 C CNN
-F 4 "RTC" H 4095 4430 50  0001 C CNN "Optional"
+F 4 "RTC" H 4095 4430 50  0001 C CNN "Section"
 	1    4095 4430
 	-1   0    0    1
@@
 F 2 "Diode_THT:D_DO-35_SOD27_P12.70mm_Horizontal" H 3365 5100 50  0001 C CNN
 F 3 "~" H 3365 5100 50  0001 C CNN
-F 4 "RTC" H 3365 5100 50  0001 C CNN "Optional"
+F 4 "RTC" H 3365 5100 50  0001 C CNN "Section"
 	1    3365 5100
 	-1   0    0    1
