File: trapdoor.sch (KiCad schematic (older format))
At the start: 2 parts, among them P9 TRAPDOOR

Commit message: Begin adding part numbers
Parts:
- JP7A1: MFG Name (none) -> SKIP; MFG Part Num (none) -> SKIP; Optional (none) -> JMP
- P9: Optional (none) -> CONN
Changed lines of the file:
@@
 F 2 "Raemixx500:Trapdoor" H 6155 3730 50  0001 C CNN
 F 3 "DOCUMENTATION" H 6155 3730 50  0001 C CNN
+F 4 "CONN" H 6155 3730 50  0001 C CNN "Optional"
 	1    6155 3730
 	1    0    0    -1
@@
 F 2 "Raemixx500:Jumper3-Open" H 9705 4200 50  0001 C CNN
 F 3 "~" H 9705 4200 50  0001 C CNN
+F 4 "SKIP" H 9705 4200 50  0001 C CNN "MFG Name"
+F 5 "SKIP" H 9705 4200 50  0001 C CNN "MFG Part Num"
+F 6 "JMP" H 9705 4200 50  0001 C CNN "Optional"
 	1    9705 4200
 	0    -1   -1   0

Commit message: Rename "Optional" Field to "Section"
Parts:
- JP7A1: Optional JMP -> (none); Section (none) -> JMP
- P9: Optional CONN -> (none); Section (none) -> CONN
Changed lines of the file:
@@
 F 2 "Raemixx500:Trapdoor" H 6155 3730 50  0001 C CNN
 F 3 "DOCUMENTATION" H 6155 3730 50  0001 C CNN
-F 4 "CONN" H 6155 3730 50  0001 C CNN "Optional"
+F 4 "CONN" H 6155 3730 50  0001 C CNN "Section"
 	1    6155 3730
 	1    0    0    -1
@@
 F 4 "SKIP" H 9705 4200 50  0001 C CNN "MFG Name"
 F 5 "SKIP" H 9705 4200 50  0001 C CNN "MFG Part Num"
-F 6 "JMP" H 9705 4200 50  0001 C CNN "Optional"
+F 6 "JMP" H 9705 4200 50  0001 C CNN "Section"
 	1    9705 4200
 	0    -1   -1   0
